Commit message: Modificación de los nobres del urdf de robotino

File: urdf/robotino/robotino.urdf.xacro (robot description, xacro)
@@ -3,9 +3,9 @@
   <!-- ==================== Properties ==================== -->
   <xacro:property name="mesh_scale"   value="0.01 0.01 0.01"/>
-  <xacro:property name="wheel_mesh"   value="package://robotino_description/model/Robotino3_SplitWheel.dae"/>
-  <xacro:property name="body_mesh"    value="package://robotino_description/model/Robotino3_SplitMain_NoCamera.dae"/>
-  <xacro:property name="tower_mesh"   value="package://robotino_description/model/Robotino3_Platform.dae"/>
-  <xacro:property name="hokuyo_mesh"  value="package://robotino_description/meshes/sensors/hokuyo.dae"/>
-  <xacro:property name="kinect_mesh"  value="package://robotino_description/meshes/sensors/kinect.dae"/>
+  <xacro:property name="wheel_mesh"   value="package://justina_descritpion/model/robotino/Robotino3_SplitWheel.dae"/>
+  <xacro:property name="body_mesh"    value="package://justina_descritpion/model/robotino/Robotino3_SplitMain_NoCamera.dae"/>
+  <xacro:property name="tower_mesh"   value="package://justina_descritpion/model/robotino/Robotino3_Platform.dae"/>
+  <xacro:property name="hokuyo_mesh"  value="package://justina_descritpion/meshes/robotino/sensors/hokuyo.dae"/>
+  <xacro:property name="kinect_mesh"  value="package://justina_descritpion/meshes/robotino/sensors/kinect.dae"/>
   <!-- ==================== Macros ==================== -->
   <xacro:macro name="wheel_link" params="index xyz rpy">

Commit message: repair xacro

File: urdf/robotino/robotino.urdf.xacro (robot description, xacro)
@@ -3,9 +3,9 @@
   <!-- ==================== Properties ==================== -->
   <xacro:property name="mesh_scale"   value="0.01 0.01 0.01"/>
-  <xacro:property name="wheel_mesh"   value="package://justina_descritpion/model/robotino/Robotino3_SplitWheel.dae"/>
-  <xacro:property name="body_mesh"    value="package://justina_descritpion/model/robotino/Robotino3_SplitMain_NoCamera.dae"/>
-  <xacro:property name="tower_mesh"   value="package://justina_descritpion/model/robotino/Robotino3_Platform.dae"/>
-  <xacro:property name="hokuyo_mesh"  value="package://justina_descritpion/meshes/robotino/sensors/hokuyo.dae"/>
-  <xacro:property name="kinect_mesh"  value="package://justina_descritpion/meshes/robotino/sensors/kinect.dae"/>
+  <xacro:property name="wheel_mesh"   value="package://justina_description/model/robotino/Robotino3_SplitWheel.dae"/>
+  <xacro:property name="body_mesh"    value="package://justina_description/model/robotino/Robotino3_SplitMain_NoCamera.dae"/>
+  <xacro:property name="tower_mesh"   value="package://justina_description/model/robotino/Robotino3_Platform.dae"/>
+  <xacro:property name="hokuyo_mesh"  value="package://justina_description/meshes/robotino/sensors/hokuyo.dae"/>
+  <xacro:property name="kinect_mesh"  value="package://justina_description/meshes/robotino/sensors/kinect.dae"/>
   <!-- ==================== Macros ==================== -->
   <xacro:macro name="wheel_link" params="index xyz rpy">
