Commit message: references in xacro amend

File: urdf/robotino/jestino_base.urdf.xacro (robot description, xacro)
@@ -7,10 +7,10 @@
         <origin xyz="0 0 0" rpy="0 0 0"/>
         <geometry>
-          <mesh filename="package://justina_description/model/Robotino3_SplitWheel.dae" scale="0.01 0.01 0.01"/>
+          <mesh filename="package://justina_description/model/robotino/Robotino3_SplitWheel.dae" scale="0.01 0.01 0.01"/>
         </geometry>
       </visual>
       <collision>
         <geometry>
-          <mesh filename="package://justina_description/model/Robotino3_SplitWheel.dae" scale="0.01 0.01 0.01"/>
+          <mesh filename="package://justina_description/model/robotino/Robotino3_SplitWheel.dae" scale="0.01 0.01 0.01"/>
         </geometry>
       </collision>
@@ -28,5 +28,5 @@
       <origin xyz="0 0 0.035" rpy="0 0 1.5707"/>
       <geometry>
-        <mesh filename="package://justina_description/model/Robotino3_SplitMain_NoCamera.dae" scale="0.01 0.01 0.01"/>
+        <mesh filename="package://justina_description/model/robotino/Robotino3_SplitMain_NoCamera.dae" scale="0.01 0.01 0.01"/>
       </geometry>
     </visual>
@@ -34,5 +34,5 @@
       <origin xyz="0 0 0.035" rpy="0 0 1.5707"/>
       <geometry>
-        <mesh filename="package://justina_description/model/Robotino3_SplitMain_NoCamera.dae" scale="0.01 0.01 0.01"/>
+        <mesh filename="package://justina_description/model/robotino/Robotino3_SplitMain_NoCamera.dae" scale="0.01 0.01 0.01"/>
       </geometry>
     </collision>
@@ -98,5 +98,5 @@
     <visual>
       <geometry>
-        <mesh filename="package://robotino_description/meshes/sensors/hokuyo.dae" scale="0.01 0.01 0.01"/>
+        <mesh filename="package://justina_description/meshes/robotino/sensors/hokuyo.dae" scale="0.01 0.01 0.01"/>
       </geometry>
       <origin xyz="0 0 -0.055" rpy="0 0 1.57"/>
@@ -104,5 +104,5 @@
     <collision>
       <geometry>
-        <mesh filename="package://robotino_description/meshes/sensors/hokuyo.dae" scale="0.01 0.01 0.01"/>
+        <mesh filename="package://justina_description/meshes/robotino/sensors/hokuyo.dae" scale="0.01 0.01 0.01"/>
       </geometry>
       <origin xyz="0 0 -0.055" rpy="0 0 1.57"/>
