Commit message: justina urdf update

File: urdf/justina/justina.urdf (robot description, URDF)
Before this commit: robot justina, 28 links, 27 joints
Links:
- link arm: geometry collision mesh filename=package://justina_description/meshes/justina/arm/arm.dae; collision mesh filename=package://justina_description/meshes/justina/servos/Mx64.dae
- link base_link: geometry collision mesh filename=package://justina_description/model/robotino/Robotino3_Spli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 scale=0.01 0.01 0.01; visual mesh filename=package://justina_description/model/robotino/Robotino3_Spli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 scale=0.01 0.01 0.01
- link camera_link: geometry collision box size=0.029 0.103 0.02; visual mesh filename=package://justina_description/meshes/robotino/sensors/kinec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 scale=1 1 1
- link forearm: geometry collision mesh filename=package://justina_description/meshes/justina/arm/forearm.dae; collision mesh filename=package://justina_description/meshes/justina/servos/Mx106.d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
- link gripper_motors: geometry collision mesh filename=package://justina_description/meshes/justina/servos/Mx28-2.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; visual mesh filename=package://justina_description/meshes/justina/servos/Mx28-2.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
- link head_link1: geometry collision box size=0.06 0.04 0.04; visual mesh filename=package://justina_description/meshes/justina/servos/Mx64.dae
- link head_link2: geometry collision box size=0.04 0.04 0.06; visual mesh filename=package://justina_description/meshes/justina/servos/Mx64.dae
- link laser_link: geometry collision mesh filename=package://justina_description/meshes/robotino/sensors/hokuy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 scale=0.01 0.01 0.01; visual mesh filename=package://justina_description/meshes/robotino/sensors/hokuy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 scale=0.01 0.01 0.01
- link left_arm: geometry collision mesh filename=package://justina_description/meshes/justina/arm/arm.dae; collision mesh filename=package://justina_description/meshes/justina/servos/Mx64.dae
- link left_forearm: geometry collision mesh filename=package://justina_description/meshes/justina/arm/forearm.dae; collision mesh filename=package://justina_description/meshes/justina/servos/Mx106.d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
- link left_gripper_motors: geometry collision mesh filename=package://justina_description/meshes/justina/servos/Mx28-2.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; visual mesh filename=package://justina_description/meshes/justina/servos/Mx28-2.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
- link left_jaw: geometry collision mesh filename=package://justina_description/meshes/justina/arm/gripper.dae; visual mesh filename=package://justina_description/meshes/justina/arm/gripper.dae
- link left_left_jaw: geometry collision mesh filename=package://justina_description/meshes/justina/arm/gripper.dae; visual mesh filename=package://justina_description/meshes/justina/arm/gripper.dae
- link left_right_jaw: geometry collision mesh filename=package://justina_description/meshes/justina/arm/gripper.dae; visual mesh filename=package://justina_description/meshes/justina/arm/gripper.dae
- link left_shoulder_frame: geometry collision mesh filename=package://justina_description/meshes/justina/arm/shoulder_f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; visual mesh filename=package://justina_description/meshes/justina/arm/shoulder_f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
- link neck_link: geometry collision box size=0.02 0.02 0.02; visual mesh filename=package://justina_description/meshes/justina/head/careta.dae
- link right_jaw: geometry collision mesh filename=package://justina_description/meshes/justina/arm/gripper.dae; visual mesh filename=package://justina_description/meshes/justina/arm/gripper.dae
- link shoulder_frame: geometry collision mesh filename=package://justina_description/meshes/justina/arm/shoulder_f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; visual mesh filename=package://justina_description/meshes/justina/arm/shoulder_f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
- link shoulders_left_link: geometry collision mesh filename=package://justina_description/meshes/justina/servos/Mx106-2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; visual mesh filename=package://justina_description/meshes/justina/servos/Mx106-2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
- link shoulders_right_link: geometry collision mesh filename=package://justina_description/meshes/justina/servos/Mx106-2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; visual mesh filename=package://justina_description/meshes/justina/servos/Mx106-2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
- link torso_link: geometry collision mesh filename=package://justina_description/meshes/justina/torso/justina_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; visual mesh filename=package://justina_description/meshes/justina/torso/justina_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
- link wheel0_link: geometry collision mesh filename=package://justina_description/model/robotino/Robotino3_Spli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 scale=0.01 0.01 0.01; visual mesh filename=package://justina_description/model/robotino/Robotino3_Spli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 scale=0.01 0.01 0.01
- link wheel1_link: geometry collision mesh filename=package://justina_description/model/robotino/Robotino3_Spli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 scale=0.01 0.01 0.01; visual mesh filename=package://justina_description/model/robotino/Robotino3_Spli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 scale=0.01 0.01 0.01
- link wheel2_link: geometry collision mesh filename=package://justina_description/model/robotino/Robotino3_Spli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 scale=0.01 0.01 0.01; visual mesh filename=package://justina_description/model/robotino/Robotino3_Spli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 scale=0.01 0.01 0.01
