Commit message: justina upper model

File: urdf/justina/components/justina_head.xacro (robot description, xacro)
@@ -1,10 +1,10 @@
 <?xml version="1.0"?>
 <robot name="justina_head" xmlns:xacro="http://www.ros.org/wiki/xacro">
-  <xacro:include filename="$(find justina_description)/urdf/components/justina_head.gazebo"/>
+  <xacro:include filename="$(find justina_description)/urdf/justina/components/justina_head.gazebo"/>
   <!--HEAD LINKS AND JOINTS-->
   <link name="head_link1">
     <visual>
       <origin xyz= "-0.01 0 0.03" rpy="0 0 -1.5707"/>
-      <geometry><mesh filename="package://justina_description/meshes/servos/Mx64.dae"/></geometry>
+      <geometry><mesh filename="package://justina_description/meshes/justina/servos/Mx64.dae"/></geometry>
       <material name="blue"/>
     </visual>
@@ -23,5 +23,5 @@
       <origin xyz= "-0.01 0.0 0.06" rpy="1.5707 0 0"/>
       <geometry>
-        <mesh filename="package://justina_description/meshes/servos/Mx64.dae"/>
+        <mesh filename="package://justina_description/meshes/justina/servos/Mx64.dae"/>
       </geometry>
       <material name="orange"/>
@@ -52,5 +52,5 @@
       <geometry>
         <!--box size="0.02 0.02 0.02"/-->
-        <mesh filename="package://justina_description/meshes/head/careta.dae"/>
+        <mesh filename="package://justina_description/meshes/justina/head/careta.dae"/>
       </geometry>
       <material name="black"/>
@@ -81,5 +81,5 @@
       <geometry>
         <!--box size=" 0.029 0.103 0.02"/-->
-        <mesh filename="package://robotino_description/meshes/sensors/kinect.dae" scale="1 1 1"/>
+        <mesh filename="package://justina_description/meshes/robotino/sensors/kinect.dae" scale="1 1 1"/>
       </geometry>
       <material name="gray"/>

File: urdf/justina/components/justina_left_arm.xacro (robot description, xacro)
@@ -1,5 +1,5 @@
 <?xml version="1.0"?>
 <robot name="justina_left_arm" xmlns:xacro="http://www.ros.org/wiki/xacro">
-  <!--xacro:include filename="$(find justina_description)/urdf/components/justina_left_arm.gazebo"/-->
+  <!--xacro:include filename="$(find justina_description)/urdf/justina/components/justina_left_arm.gazebo"/-->
   <!-- LEFT ARM LINKS -->
   <link name="shoulders_left_link">
@@ -7,5 +7,5 @@
       <origin xyz="0 -0.01 0.02" rpy = "0 3.1415 0"/>
       <geometry>
-        <mesh filename="package://justina_description/meshes/servos/Mx106-2.dae"/>
+        <mesh filename="package://justina_description/meshes/justina/servos/Mx106-2.dae"/>
       </geometry>
     </visual>
@@ -13,5 +13,5 @@
       <origin xyz="0 -0.01 0.02" rpy = "0 3.1415 0"/>
       <geometry>
-        <mesh filename="package://justina_description/meshes/servos/Mx106-2.dae"/>
+        <mesh filename="package://justina_description/meshes/justina/servos/Mx106-2.dae"/>
       </geometry>
     </collision>
@@ -29,5 +29,5 @@
       <origin xyz="0 -0.01 0.01" rpy="0 0 -1.5707"/>
       <geometry>
-       <mesh filename="package://justina_description/meshes/arm/shoulder_frame.dae"/>
+       <mesh filename="package://justina_description/meshes/justina/arm/shoulder_frame.dae"/>
       </geometry>
       <material name = "la_material"><color rgba="1.0 0.5 0 1"/></material>
@@ -36,5 +36,5 @@
       <origin xyz="0 -0.01 0.01" rpy="0 0 -1.5707"/>
       <geometry>
-       <mesh filename="package://justina_description/meshes/arm/shoulder_frame.dae"/>
+       <mesh filename="package://justina_description/meshes/justina/arm/shoulder_frame.dae"/>
       </geometry>
     </collision>
@@ -52,5 +52,5 @@
       <origin xyz="0 0 -0.02" rpy="0 0 6.2822"/>
       <geometry>
-       <mesh filename="package://justina_description/meshes/servos/Mx64.dae"/>
+       <mesh filename="package://justina_description/meshes/justina/servos/Mx64.dae"/>
       </geometry>
     </visual>
@@ -58,5 +58,5 @@
       <origin xyz="0 0 -0.216" rpy="0 3.1416 1.5707"/>
       <geometry>
-       <mesh filename="package://justina_description/meshes/arm/arm.dae"/>
+       <mesh filename="package://justina_description/meshes/justina/arm/arm.dae"/>
       </geometry>
     </visual>
@@ -64,5 +64,5 @@
       <origin xyz="0 0 -0.02" rpy="0 0 6.2822"/>
       <geometry>
-       <mesh filename="package://justina_description/meshes/servos/Mx64.dae"/>
+       <mesh filename="package://justina_description/meshes/justina/servos/Mx64.dae"/>
       </geometry>
     </collision>
@@ -70,5 +70,5 @@
       <origin xyz="0 0 -0.216" rpy="0 3.1416 1.5707"/>
       <geometry>
-       <mesh filename="package://justina_description/meshes/arm/arm.dae"/>
+       <mesh filename="package://justina_description/meshes/justina/arm/arm.dae"/>
       </geometry>
     </collision>
@@ -86,5 +86,5 @@
       <origin xyz="0 0 0" rpy="1.5707 0 0"/>
       <geometry>
-       <mesh filename="package://justina_description/meshes/servos/Mx106.dae"/>
+       <mesh filename="package://justina_description/meshes/justina/servos/Mx106.dae"/>
       </geometry>
     </visual>
@@ -92,5 +92,5 @@
       <origin xyz="0 0 -0.12" rpy="0 0 1.5707"/>
       <geometry>
-       <mesh filename="package://justina_description/meshes/arm/forearm.dae"/>
+       <mesh filename="package://justina_description/meshes/justina/arm/forearm.dae"/>
       </geometry>
     </visual>
@@ -98,5 +98,5 @@
       <origin xyz="0.009 0.001 -0.21" rpy="0 0 -1.5707"/>
       <geometry>
-       <mesh filename="package://justina_description/meshes/servos/Mx64.dae"/>
+       <mesh filename="package://justina_description/meshes/justina/servos/Mx64.dae"/>
       </geometry>
     </visual>
@@ -104,5 +104,5 @@
       <origin xyz="0 0 0" rpy="0 0 0"/>
       <geometry>
-       <mesh filename="package://justina_description/meshes/servos/Mx106.dae"/>
+       <mesh filename="package://justina_description/meshes/justina/servos/Mx106.dae"/>
       </geometry>
     </collision>
@@ -110,5 +110,5 @@
       <origin xyz="0 0 -0.12" rpy="0 0 1.5707"/>
       <geometry>
-       <mesh filename="package://justina_description/meshes/arm/forearm.dae"/>
+       <mesh filename="package://justina_description/meshes/justina/arm/forearm.dae"/>
       </geometry>
     </collision>
@@ -116,5 +116,5 @@
       <origin xyz="0.009 0.001 -0.21" rpy="0 0 -1.5707"/>
       <geometry>
-       <mesh filename="package://justina_description/meshes/servos/Mx64.dae"/>
+       <mesh filename="package://justina_description/meshes/justina/servos/Mx64.dae"/>
       </geometry>
     </collision>
@@ -132,5 +132,5 @@
       <origin xyz="0 -0.004 0" rpy="1.5707 -1.5707 0"/>
       <geometry>
-        <mesh filename="package://justina_description/meshes/servos/Mx28-2.dae"/>
+        <mesh filename="package://justina_description/meshes/justina/servos/Mx28-2.dae"/>
       </geometry>
     </visual>
@@ -138,5 +138,5 @@
       <origin xyz="0 -0.004 0" rpy="1.5707 -1.5707 0"/>
       <geometry>
-        <mesh filename="package://justina_description/meshes/servos/Mx28-2.dae"/>
+        <mesh filename="package://justina_description/meshes/justina/servos/Mx28-2.dae"/>
       </geometry>
     </collision>
@@ -154,5 +154,5 @@
       <origin xyz="0 0 0" rpy="0 1.5707 3.1416"/>
       <geometry>
-        <mesh filename="package://justina_description/meshes/arm/gripper.dae"/>
+        <mesh filename="package://justina_description/meshes/justina/arm/gripper.dae"/>
       </geometry>
     </visual>
@@ -160,5 +160,5 @@
       <origin xyz="0 0 0" rpy="0 1.5707 3.1416"/>
       <geometry>
-        <mesh filename="package://justina_description/meshes/arm/gripper.dae"/>
+        <mesh filename="package://justina_description/meshes/justina/arm/gripper.dae"/>
       </geometry>
     </collision>
@@ -176,5 +176,5 @@
       <origin xyz="0 0 0" rpy="0 1.5707 0"/>
       <geometry>
-        <mesh filename="package://justina_description/meshes/arm/gripper.dae"/>
+        <mesh filename="package://justina_description/meshes/justina/arm/gripper.dae"/>
       </geometry>
     </visual>
@@ -182,5 +182,5 @@
       <origin xyz="0 0 0" rpy="0 0 0"/>
       <geometry>
-        <mesh filename="package://justina_description/meshes/arm/gripper.dae"/>
+        <mesh filename="package://justina_description/meshes/justina/arm/gripper.dae"/>
       </geometry>
     </collision>

File: urdf/justina/components/justina_right_arm.xacro (robot description, xacro)
@@ -1,5 +1,5 @@
 <?xml version="1.0"?>
 <robot name="justina_right_arm" xmlns:xacro="http://www.ros.org/wiki/xacro">
-  <!--xacro:include filename="$(find justina_description)/urdf/components/justina_right_arm.gazebo"/-->
+  <!--xacro:include filename="$(find justina_description)/urdf/justina/components/justina_right_arm.gazebo"/-->
   <!-- RIGHT ARM LINKS -->
   <link name="shoulders_right_link">
@@ -7,5 +7,5 @@
       <origin xyz="0 -0.01 0.02" rpy = "0 3.1415 0"/>
       <geometry>
-        <mesh filename="package://justina_description/meshes/servos/Mx106-2.dae"/>
+        <mesh filename="package://justina_description/meshes/justina/servos/Mx106-2.dae"/>
       </geometry>
     </visual>
@@ -13,5 +13,5 @@
       <origin xyz="0 -0.01 0.02" rpy = "0 3.1415 0"/>
       <geometry>
-        <mesh filename="package://justina_description/meshes/servos/Mx106-2.dae"/>
+        <mesh filename="package://justina_description/meshes/justina/servos/Mx106-2.dae"/>
       </geometry>
     </collision>
@@ -29,5 +29,5 @@
       <origin xyz="0 -0.01 0.01" rpy="0 0 -1.5707"/>
       <geometry>
-       <mesh filename="package://justina_description/meshes/arm/shoulder_frame.dae"/>
+       <mesh filename="package://justina_description/meshes/justina/arm/shoulder_frame.dae"/>
       </geometry>
       <material name = "la_material"><color rgba="1.0 0.5 0 1"/></material>
@@ -36,5 +36,5 @@
       <origin xyz="0 -0.01 0.01" rpy="0 0 -1.5707"/>
       <geometry>
-       <mesh filename="package://justina_description/meshes/arm/shoulder_frame.dae"/>
+       <mesh filename="package://justina_description/meshes/justina/arm/shoulder_frame.dae"/>
       </geometry>
     </collision>
@@ -52,5 +52,5 @@
       <origin xyz="0 0 -0.02" rpy="0 0 3.1416"/>
       <geometry>
-       <mesh filename="package://justina_description/meshes/servos/Mx64.dae"/>
+       <mesh filename="package://justina_description/meshes/justina/servos/Mx64.dae"/>
       </geometry>
     </visual>
@@ -58,5 +58,5 @@
       <origin xyz="0 0 -0.216" rpy="0 3.1416 -1.5707"/>
       <geometry>
-       <mesh filename="package://justina_description/meshes/arm/arm.dae"/>
+       <mesh filename="package://justina_description/meshes/justina/arm/arm.dae"/>
       </geometry>
     </visual>
@@ -64,5 +64,5 @@
       <origin xyz="0 0 -0.02" rpy="0 0 3.1416"/>
       <geometry>
-       <mesh filename="package://justina_description/meshes/servos/Mx64.dae"/>
+       <mesh filename="package://justina_description/meshes/justina/servos/Mx64.dae"/>
       </geometry>
     </collision>
@@ -70,5 +70,5 @@
       <origin xyz="0 0 -0.216" rpy="0 3.1416 -1.5707"/>
       <geometry>
-       <mesh filename="package://justina_description/meshes/arm/arm.dae"/>
+       <mesh filename="package://justina_description/meshes/justina/arm/arm.dae"/>
       </geometry>
     </collision>
@@ -86,5 +86,5 @@
       <origin xyz="0 0 0" rpy="1.5707 0 0"/>
       <geometry>
-       <mesh filename="package://justina_description/meshes/servos/Mx106.dae"/>
+       <mesh filename="package://justina_description/meshes/justina/servos/Mx106.dae"/>
       </geometry>
     </visual>
@@ -92,5 +92,5 @@
       <origin xyz="0 0 -0.12" rpy="0 0 1.5707"/>
       <geometry>
-       <mesh filename="package://justina_description/meshes/arm/forearm.dae"/>
+       <mesh filename="package://justina_description/meshes/justina/arm/forearm.dae"/>
       </geometry>
     </visual>
@@ -98,5 +98,5 @@
       <origin xyz="0.009 0.001 -0.21" rpy="0 0 -1.5707"/>
       <geometry>
-       <mesh filename="package://justina_description/meshes/servos/Mx64.dae"/>
+       <mesh filename="package://justina_description/meshes/justina/servos/Mx64.dae"/>
       </geometry>
     </visual>
@@ -104,5 +104,5 @@
       <origin xyz="0 0 0" rpy="0 0 0"/>
       <geometry>
-       <mesh filename="package://justina_description/meshes/servos/Mx106.dae"/>
+       <mesh filename="package://justina_description/meshes/justina/servos/Mx106.dae"/>
       </geometry>
     </collision>
@@ -110,5 +110,5 @@
       <origin xyz="0 0 -0.12" rpy="0 0 1.5707"/>
       <geometry>
-       <mesh filename="package://justina_description/meshes/arm/forearm.dae"/>
+       <mesh filename="package://justina_description/meshes/justina/arm/forearm.dae"/>
       </geometry>
     </collision>
@@ -116,5 +116,5 @@
       <origin xyz="0.009 0.001 -0.21" rpy="0 0 -1.5707"/>
       <geometry>
-       <mesh filename="package://justina_description/meshes/servos/Mx64.dae"/>
+       <mesh filename="package://justina_description/meshes/justina/servos/Mx64.dae"/>
       </geometry>
     </collision>
@@ -132,5 +132,5 @@
       <origin xyz="0 -0.004 0" rpy="1.5707 -1.5707 0"/>
       <geometry>
-        <mesh filename="package://justina_description/meshes/servos/Mx28-2.dae"/>
+        <mesh filename="package://justina_description/meshes/justina/servos/Mx28-2.dae"/>
       </geometry>
     </visual>
@@ -138,5 +138,5 @@
       <origin xyz="0 -0.004 0" rpy="1.5707 -1.5707 0"/>
       <geometry>
-        <mesh filename="package://justina_description/meshes/servos/Mx28-2.dae"/>
+        <mesh filename="package://justina_description/meshes/justina/servos/Mx28-2.dae"/>
       </geometry>
     </collision>
@@ -154,5 +154,5 @@
       <origin xyz="0 0 0" rpy="0 1.5707 3.1416"/>
       <geometry>
-        <mesh filename="package://justina_description/meshes/arm/gripper.dae"/>
+        <mesh filename="package://justina_description/meshes/justina/arm/gripper.dae"/>
       </geometry>
     </visual>
@@ -160,5 +160,5 @@
       <origin xyz="0 0 0" rpy="0 1.5707 3.1416"/>
       <geometry>
-        <mesh filename="package://justina_description/meshes/arm/gripper.dae"/>
+        <mesh filename="package://justina_description/meshes/justina/arm/gripper.dae"/>
       </geometry>
     </collision>
@@ -176,5 +176,5 @@
       <origin xyz="0 0 0" rpy="0 1.5707 0"/>
       <geometry>
-        <mesh filename="package://justina_description/meshes/arm/gripper.dae"/>
+        <mesh filename="package://justina_description/meshes/justina/arm/gripper.dae"/>
       </geometry>
     </visual>
@@ -182,5 +182,5 @@
       <origin xyz="0 0 0" rpy="0 0 0"/>
       <geometry>
-        <mesh filename="package://justina_description/meshes/arm/gripper.dae"/>
+        <mesh filename="package://justina_description/meshes/justina/arm/gripper.dae"/>
       </geometry>
     </collision>

File: urdf/justina/components/justina_torso.xacro (robot description, xacro)
@@ -1,5 +1,5 @@
 <?xml version="1.0"?>
 <robot name="justina_torso" xmlns:xacro="http://www.ros.org/wiki/xacro">
-<!--xacro:include filename="$(find justina_description)/urdf/justina_torso.gazebo"/-->
+<!--xacro:include filename="$(find justina_description)/urdf/justina/justina_torso.gazebo"/-->
   <xacro:macro name="box_inertia" params="m x y z">
     <inertia  ixx="${m*(y*y+z*z)/12}" ixy = "0" ixz = "0" iyy="${m*(x*x+z*z)/12}" iyz = "0" izz="${m*(x*x+z*z)/12}"/>
@@ -13,5 +13,5 @@
       <origin xyz= "0.0 0.0 -0.1" rpy="0 0 0"/>
       <geometry>
-	    <mesh filename="package://justina_description/meshes/torso/justina_chest.dae"/>
+	    <mesh filename="package://justina_description/meshes/justina/torso/justina_chest.dae"/>
       </geometry>
     </collision>
@@ -20,5 +20,5 @@
       <!--origin xyz= "0.04 -0.097 -0.55" rpy="0 0 0"/-->
       <geometry>
-	    <mesh filename="package://justina_description/meshes/torso/justina_chest.dae"/>
+	    <mesh filename="package://justina_description/meshes/justina/torso/justina_chest.dae"/>
       </geometry>
       <material name="black_gray"><color rgba="0.2 0.2 0.2 1"/></material>

File: urdf/justina/justina.xacro (robot description, xacro)
@@ -1,11 +1,11 @@
 <?xml version="1.0"?>
 <robot name="justina" xmlns:xacro="http://www.ros.org/wiki/xacro">
-  <xacro:include filename="$(find justina_description)/urdf/macros.xacro"/>
-  <xacro:include filename="$(find justina_description)/urdf/materials.xacro"/>
-  <xacro:include filename="$(find robotino_description)/urdf/jestino_base.urdf.xacro"/>
-  <xacro:include filename="$(find justina_description)/urdf/components/justina_torso.xacro"/>
-  <xacro:include filename="$(find justina_description)/urdf/components/justina_left_arm.xacro"/>
-  <xacro:include filename="$(find justina_description)/urdf/components/justina_right_arm.xacro"/>
-  <xacro:include filename="$(find justina_description)/urdf/components/justina_head.xacro"/>
+  <xacro:include filename="$(find justina_description)/urdf/justina/macros.xacro"/>
+  <xacro:include filename="$(find justina_description)/urdf/justina/materials.xacro"/>
+  <xacro:include filename="$(find justina_description)/urdf/robotino/jestino_base.urdf.xacro"/>
+  <xacro:include filename="$(find justina_description)/urdf/justina/components/justina_torso.xacro"/>
+  <xacro:include filename="$(find justina_description)/urdf/justina/components/justina_left_arm.xacro"/>
+  <xacro:include filename="$(find justina_description)/urdf/justina/components/justina_right_arm.xacro"/>
+  <xacro:include filename="$(find justina_description)/urdf/justina/components/justina_head.xacro"/>
   <joint name="torso_connect" type="fixed">
     <origin xyz= "0.0 0.0 0.80" rpy="0 0 0"/>

Commit message: update repo for camera_link

File: urdf/justina/components/justina_head.xacro (robot description, xacro)
@@ -78,5 +78,5 @@
   <link name="camera_link">
     <visual>
-      <origin xyz="0 0 0" rpy="0 0 1.5707"/>
+      <origin xyz="0 0 0" rpy="-1.5707 0 3.1415"/>
       <geometry>
         <!--box size=" 0.029 0.103 0.02"/-->
@@ -98,5 +98,5 @@
   </link>
   <joint name="camera_link_connect" type="fixed">
-    <origin xyz="0 0 0.065" rpy="0 0 0"/>
+    <origin xyz="0 0 0.065" rpy="-1.5707 0 -1.5707"/>
     <parent link="neck_link"/>
     <child link="camera_link"/>
