Commit message: Virtual justina: edit mesh to match real robot dimensions, rename links and joints in both arms, add new colliders

File: urdf/justina_gazebo/festina_base_low_poly.xacro (robot description, xacro)
@@ -1,5 +1,5 @@
 <?xml version="1.0"?>
 <robot name="robotino" xmlns:xacro="http://www.ros.org/wiki/xacro">
-    <xacro:property name="M_PI" value="3.1415926535897931" />
+    <!-- NOTE Wheels have 0.01 offset from ground to match with visual texture floor in LAB world -->
     <!-- Base Robotino -->
     <link name="base_link">
@@ -7,8 +7,8 @@
             <mass value="10.0"/>
             <inertia ixx="0.1" ixy="0.0" ixz="0.0" iyy="0.1" iyz="0.0" izz="0.1"/>
-            <origin xyz="0 0 0.035" rpy="0 0 0"/>
+            <origin xyz="0 0 0" rpy="0 0 0"/>
         </inertial>
         <visual>
-            <origin xyz="0 0 0" rpy="0 0 ${M_PI/2}"/>
+            <origin xyz="0 0 -0.03" rpy="0 0 0"/>
             <geometry>
                 <mesh filename="package://justina_description/meshes/robotino_low_poly/Robotino3_LowPoly.dae" scale="1 1 1"/>
@@ -16,7 +16,7 @@
         </visual>
         <collision>
-            <origin xyz="0 0 0.085" rpy="0 0 0"/>
+            <origin xyz="0 0 -0.03" rpy="0 0 0"/>
             <geometry>
-                <cylinder radius="0.234" length="0.2"/>
+                <mesh filename="package://justina_description/meshes/robotino_low_poly/Robotino3_Collider_LowPoly.dae" scale="1 1 1"/>
             </geometry>
         </collision>
@@ -78,5 +78,5 @@
         </visual>
         <collision>
-            <origin xyz="0 0 0.035" rpy="0 0 0"/>
+            <origin xyz="0 0 0.0" rpy="0 0 0"/>
             <geometry>
                 <box size="0.05 0.05 0.07"/>
@@ -97,5 +97,5 @@
         </inertial>
         <visual>
-            <origin xyz="0 0 0.0" rpy="0 0 ${M_PI/2}"/>
+            <origin xyz="0 0 0" rpy="0 0 0"/>
             <geometry>
                 <mesh filename="package://justina_description/meshes/robotino_low_poly/Justina_Platform_LowPoly.dae" scale="1 1 1"/>
@@ -103,5 +103,5 @@
         </visual>
         <collision>
-            <origin xyz="0 0 0.413" rpy="0 0 0"/>
+            <origin xyz="0 0 0.49" rpy="0 0 0"/>
             <geometry>
                 <cylinder radius="0.075" length="0.59"/>
@@ -109,8 +109,9 @@
         </collision>
     </link>
+    <!-- tower have an offset of 0.06 -->
     <joint name="tower_joint" type="fixed">
         <parent link="base_link"/>
         <child link="tower_link"/>
-        <origin xyz="0 0 0.06" rpy="0 0 0"/>
+        <origin xyz="0 0 -0.05" rpy="0 0 0"/>
     </joint>
 </robot>

File: urdf/justina_gazebo/justina.xacro (robot description, xacro)
@@ -1,4 +1,5 @@
 <?xml version="1.0"?>
 <robot name="justina" xmlns:xacro="http://www.ros.org/wiki/xacro">
+  <!-- NOTE Wheels have 0.01 offset from ground to match with visual texture floor in LAB world -->
   <xacro:include filename="$(find justina_description)/urdf/justina_gazebo/festina_base_low_poly.xacro" />
   <xacro:include filename="$(find justina_description)/urdf/justina_gazebo/justina_toso_low_poly.xacro" />
@@ -7,20 +8,20 @@
   <xacro:include filename="$(find justina_description)/urdf/justina_gazebo/justina_head_low_poly.xacro" />
   <joint name="torso_connect" type="fixed">
-    <origin xyz= "0.0 0.0 0.80" rpy="0 0 0"/>
+    <origin xyz= "0.0 0.0 0.73" rpy="0 0 0"/>
     <parent link="base_link"/>
     <child link="torso_link"/>
   </joint>
   <joint name="shoulder_left_connect" type="fixed">
-    <origin xyz="0 0.225 -0.08" rpy="0 0 0"/>
+    <origin xyz="0 0.225 -0.045" rpy="0 0 0"/>
     <parent link="spine_link"/>
-    <child link="shoulders_left_link"/>
+    <child link="left_shoulder_link"/>
   </joint>
   <joint name="shoulder_right_connect" type="fixed">
-    <origin xyz="0 -0.225 -0.08" rpy="0 0 0"/>
+    <origin xyz="0 -0.225 -0.045" rpy="0 0 0"/>
     <parent link="spine_link"/>
-    <child link="shoulders_right_link"/>
+    <child link="right_shoulder_link"/>
   </joint>
   <joint name="spine_head_connect" type="fixed">
-    <origin xyz="0 0 0.13" rpy="0 0 0"/>
+    <origin xyz="0 0 0.2" rpy="0 0 0"/>
     <parent link="spine_link"/>
     <child link="head_link1"/>

File: urdf/justina_gazebo/justina_head_low_poly.xacro (robot description, xacro)
@@ -2,4 +2,5 @@
 <robot xmlns:xacro="http://www.ros.org/wiki/xacro" name="justina">
   <!-- <xacro:include filename="$(find justina_description)/urdf/justina/components/justina_head.gazebo"/> -->
+  <xacro:property name="M_PI" value="3.1415926535897931" />
   <!--HEAD LINKS AND JOINTS-->
   <link name="head_link1">
@@ -10,33 +11,37 @@
     </inertial>
     <visual>
-      <origin xyz= "-0.01 0 0.03" rpy="0 0 -1.5707"/>
-      <geometry><mesh filename="package://justina_description/meshes/justina/servos/Servo_Mx64_LowPoly.dae"/></geometry>
+      <origin xyz= "0.0 0 0.01" rpy="0 0 -${M_PI/2}"/>
+      <geometry>
+        <mesh filename="package://justina_description/meshes/justina/servos/Servo_Mx64_LowPoly.dae" scale="1 1 1"/>
+      </geometry>
     </visual>
     <collision>
-      <origin xyz= "-0.01 0 0.03" rpy="0 0 -1.5707"/>
-      <geometry><mesh filename="package://justina_description/meshes/justina/servos/Servo_Mx64_LowPoly.dae"/></geometry>
+      <origin xyz= "0.0 0 0.01" rpy="0 0 -${M_PI/2}"/>
+      <geometry>
+        <mesh filename="package://justina_description/meshes/justina/servos/Servo_Mx64_LowPoly.dae" scale="1 1 1"/>
+      </geometry>
     </collision>
   </link>
   <link name="head_link2">
     <inertial>
-      <origin xyz="0.0 0 0.0" rpy = "0 0 0"/>
+      <origin xyz="0.0 0 0.0" rpy = "0 0 0"/>z
       <mass value = "0.15" />
       <inertia ixx = "0.00003125" iyy = "0.00003125" izz = "0.00003125" ixy = "0" ixz = "0" iyz = "0" />
     </inertial>
     <visual>
-      <origin xyz= "-0.01 0.0 0.06" rpy="1.5707 0 0"/>
+      <origin xyz= "0 0.0 0.06" rpy="${M_PI/2} 0 0"/>
       <geometry>
-        <mesh filename="package://justina_description/meshes/justina/servos/Servo_Mx64_LowPoly.dae"/>
+        <mesh filename="package://justina_description/meshes/justina/servos/Servo_Mx64_LowPoly.dae" scale="1 1 1"/>
       </geometry>
     </visual>
     <collision>
-      <origin xyz= "-0.01 0.0 0.06" rpy="1.5707 0 0"/>
+      <origin xyz= "0 0.0 0.06" rpy="${M_PI/2} 0 0"/>
       <geometry>
-        <mesh filename="package://justina_description/meshes/justina/servos/Servo_Mx64_LowPoly.dae"/>
+        <mesh filename="package://justina_description/meshes/justina/servos/Servo_Mx64_LowPoly.dae" scale="1 1 1"/>
       </geometry>
     </collision>
   </link>
   <joint name="head_pan" type="revolute">
-    <origin xyz="0.0 0 0.05" rpy="0 0 0" />
+    <origin xyz="0.0 0 0.035" rpy="0 0 0" />
     <parent link="head_link1"/>
     <child link="head_link2"/>
@@ -79,18 +84,18 @@
     </inertial>
     <visual>
-      <origin xyz="0 0 0" rpy="-1.5707 0 3.1415"/>
-      <geometry>
-        <mesh filename="package://justina_description/meshes/robotino_low_poly/sensors/kinect_LowPoly.dae" scale="1 1 1"/>
+      <origin xyz="0 0 0" rpy="0 0 0"/>
+      <geometry>camera_link
+        <mesh filename="package://justina_description/meshes/robotino_low_poly/sensors/kinect_LowPoly_B.dae" scale="1 1 1"/>
       </geometry>
     </visual>
     <collision>
-      <origin xyz= "0 0 0" rpy="-1.5707 0 3.1415"/>
+      <origin xyz= "0 0 0" rpy="0 0 0"/>
       <geometry>
-        <mesh filename="package://justina_description/meshes/robotino_low_poly/sensors/kinect_Collider.dae" scale="1 1 1"/>
+        <mesh filename="package://justina_description/meshes/robotino_low_poly/sensors/kinect_Collider_B.dae" scale="1 1 1"/>
       </geometry>
     </collision>
   </link>
   <joint name="camera_link_connect" type="fixed">
-    <origin xyz="0 0 0.065" rpy="-1.5707 0 -1.5707"/>
+    <origin xyz="0 0 0" rpy="0 0 0"/>
     <parent link="neck_link"/>
     <child link="camera_link"/>

File: urdf/justina_gazebo/justina_left_arm_low_poly.xacro (robot description, xacro)
@@ -3,5 +3,5 @@
   <!--xacro:include filename="$(find justina_description)/urdf/justina/components/justina_left_arm.gazebo"/-->
   <!-- LEFT ARM LINKS -->
-  <link name="shoulders_left_link">
+  <link name="left_shoulder_link">
     <inertial>
       <origin xyz="0 -0.01 0.02" rpy = "0 0 0"/>
@@ -12,5 +12,5 @@
       <origin xyz="0 -0.01 0.02" rpy = "0 3.1415 0"/>
       <geometry>
-        <mesh filename="package://justina_description/meshes/justina/servos/Servo_Mx106-2_LowPoly.dae"/>
+        <mesh filename="package://justina_description/meshes/justina/servos/Servo_Mx106-2_LowPoly.dae" scale="1 1 1"/>
       </geometry>
     </visual>
@@ -18,5 +18,5 @@
       <origin xyz="0 -0.01 0.02" rpy = "0 3.1415 0"/>
       <geometry>
-        <mesh filename="package://justina_description/meshes/justina/servos/Servo_Mx106-2_LowPoly.dae"/>
+        <mesh filename="package://justina_description/meshes/justina/servos/Servo_Mx106-2_LowPoly.dae" scale="1 1 1"/>
       </geometry>
     </collision>
@@ -24,18 +24,18 @@
   <link name="left_shoulder_frame">
     <inertial>
-      <origin xyz="0 -0.01 0.01" rpy = "0 0 -1.5707"/>
+      <origin xyz="0 -0.01 0.0" rpy = "0 0 -1.5707"/>
       <mass value="0.08146"/>
       <inertia ixx="0.0000813217" ixy="0.0" ixz="0.0" iyy="0.000196" iyz="0.0" izz="0.0001282"/>
     </inertial>
     <visual>
-      <origin xyz="0 -0.01 0.01" rpy="0 0 -1.5707"/>
-      <geometry>
-        <mesh filename="package://justina_description/meshes/justina/arm/Shoulder_Frame_LowPoly.dae"/>
-      </geometry>
-    </visual>
-    <collision>
-      <origin xyz="0 -0.01 0.01" rpy="0 0 -1.5707"/>
-      <geometry>
-        <mesh filename="package://justina_description/meshes/justina/arm/Shoulder_Frame_LowPoly.dae"/>
+      <origin xyz="0 -0.01 0.0" rpy="0 0 -1.5707"/>
+      <geometry>
+        <mesh filename="package://justina_description/meshes/justina/arm/Shoulder_Frame_LowPoly.dae" scale="1 1 1"/>
+      </geometry>
+    </visual>
+    <collision>
+      <origin xyz="0 -0.01 0.0" rpy="0 0 -1.5707"/>
+      <geometry>
+        <mesh filename="package://justina_description/meshes/justina/arm/Shoulder_Frame_LowPoly.dae" scale="1 1 1"/>
       </geometry>
     </collision>
@@ -50,5 +50,5 @@
       <origin xyz="0 0 -0.02" rpy="0 0 6.2822"/>
       <geometry>
-        <mesh filename="package://justina_description/meshes/justina/servos/Servo_Mx64_LowPoly.dae"/>
+        <mesh filename="package://justina_description/meshes/justina/servos/Servo_Mx64_LowPoly.dae" scale="1 1 1"/>
       </geometry>
     </visual>
@@ -56,5 +56,5 @@
       <origin xyz="0 0 -0.02" rpy="0 0 6.2822"/>
       <geometry>
-        <mesh filename="package://justina_description/meshes/justina/servos/Servo_Mx64_LowPoly.dae"/>
+        <mesh filename="package://justina_description/meshes/justina/servos/Servo_Mx64_LowPoly.dae" scale="1 1 1"/>
       </geometry>
     </collision>
@@ -62,5 +62,5 @@
       <origin xyz="0 0 -0.216" rpy="0 3.1416 1.5707"/>
       <geometry>
-        <mesh filename="package://justina_description/meshes/justina/arm/Arm_LowPoly.dae"/>
+        <mesh filename="package://justina_description/meshes/justina/arm/Arm_LowPoly.dae" scale="1 1 1"/>
       </geometry>
     </visual>
@@ -68,5 +68,5 @@
       <origin xyz="0 0 -0.216" rpy="0 3.1416 1.5707"/>
       <geometry>
-        <mesh filename="package://justina_description/meshes/justina/arm/Arm_LowPoly.dae"/>
+        <mesh filename="package://justina_description/meshes/justina/arm/Arm_LowPoly.dae" scale="1 1 1"/>
       </geometry>
     </collision>
@@ -81,5 +81,5 @@
       <origin xyz="0 0 0" rpy="1.5707 0 0"/>
       <geometry>
-        <mesh filename="package://justina_description/meshes/justina/servos/Servo_Mx106_LowPoly.dae"/>
+        <mesh filename="package://justina_description/meshes/justina/servos/Servo_Mx106_LowPoly.dae" scale="1 1 1"/>
       </geometry>
     </visual>
@@ -87,5 +87,5 @@
       <origin xyz="0 0 0" rpy="1.5707 0 0"/>
       <geometry>
-        <mesh filename="package://justina_description/meshes/justina/servos/Servo_Mx106_LowPoly.dae"/>
+        <mesh filename="package://justina_description/meshes/justina/servos/Servo_Mx106_LowPoly.dae" scale="1 1 1"/>
       </geometry>
     </collision>
@@ -93,5 +93,5 @@
       <origin xyz="0 0 -0.12" rpy="0 0 1.5707"/>
       <geometry>
-        <mesh filename="package://justina_description/meshes/justina/arm/Forearm_LowPoly.dae"/>
+        <mesh filename="package://justina_description/meshes/justina/arm/Forearm_LowPoly.dae" scale="1 1 1"/>
       </geometry>
     </visual>
@@ -99,5 +99,5 @@
       <origin xyz="0 0 -0.12" rpy="0 0 1.5707"/>
       <geometry>
-        <mesh filename="package://justina_description/meshes/justina/arm/Forearm_LowPoly.dae"/>
+        <mesh filename="package://justina_description/meshes/justina/arm/Forearm_LowPoly.dae" scale="1 1 1"/>
       </geometry>
     </collision>
@@ -105,5 +105,5 @@
       <origin xyz="0.009 0.001 -0.21" rpy="0 0 -1.5707"/>
       <geometry>
-        <mesh filename="package://justina_description/meshes/justina/servos/Servo_Mx64_LowPoly.dae"/>
+        <mesh filename="package://justina_description/meshes/justina/servos/Servo_Mx64_LowPoly.dae" scale="1 1 1"/>
       </geometry>
     </visual>
@@ -111,5 +111,5 @@
       <origin xyz="0.009 0.001 -0.21" rpy="0 0 -1.5707"/>
       <geometry>
-        <mesh filename="package://justina_description/meshes/justina/servos/Servo_Mx64_LowPoly.dae"/>
+        <mesh filename="package://justina_description/meshes/justina/servos/Servo_Mx64_LowPoly.dae" scale="1 1 1"/>
       </geometry>
     </collision>
@@ -122,17 +122,17 @@
     </inertial>
     <visual>
-      <origin xyz="0 -0.004 0" rpy="1.5707 -1.5707 0"/>
-      <geometry>
-        <mesh filename="package://justina_description/meshes/justina/servos/Servo_Mx28-2_LowPoly.dae"/>
-      </geometry>
-    </visual>
-    <collision>
-      <origin xyz="0 -0.004 0" rpy="1.5707 -1.5707 0"/>
-      <geometry>
-        <mesh filename="package://justina_description/meshes/justina/servos/Servo_Mx28-2_LowPoly.dae"/>
-      </geometry>
-    </collision>
-  </link>
-  <link name="left_right_jaw">
+      <origin xyz="0 0 0" rpy="1.5707 -1.5707 0"/>
+      <geometry>
+        <mesh filename="package://justina_description/meshes/justina/servos/Servo_Mx28-2_LowPoly.dae" scale="1 1 1"/>
+      </geometry>
+    </visual>
+    <collision>
+      <origin xyz="0 0 0" rpy="1.5707 -1.5707 0"/>
+      <geometry>
+        <mesh filename="package://justina_description/meshes/justina/servos/Servo_Mx28-2_LowPoly.dae" scale="1 1 1"/>
+      </geometry>
+    </collision>
+  </link>
+  <link name="left_jaw_right">
     <inertial>
       <origin xyz="0 0 0" rpy = "0 0 0"/>
@@ -143,5 +143,5 @@
       <origin xyz="0 0 0" rpy="0 1.5707 3.1416"/>
       <geometry>
-        <mesh filename="package://justina_description/meshes/justina/arm/Gripper_Clean.dae"/>
+        <mesh filename="package://justina_description/meshes/justina/arm/Gripper_Clean.dae" scale="1 1 1"/>
       </geometry>
     </visual>
@@ -149,9 +149,9 @@
       <origin xyz="0 0 0" rpy="0 1.5707 3.1416"/>
       <geometry>
-        <mesh filename="package://justina_description/meshes/justina/arm/Gripper_Clean.dae"/>
-      </geometry>
-    </collision>
-  </link>
-  <link name="left_left_jaw">
+        <mesh filename="package://justina_description/meshes/justina/arm/Gripper_Clean.dae" scale="1 1 1"/>
+      </geometry>
+    </collision>
+  </link>
+  <link name="left_jaw_left">
     <inertial>
       <origin xyz="0 0 0" rpy = "0 0 0"/>
@@ -162,5 +162,5 @@
       <origin xyz="0 0 0" rpy="0 1.5707 0"/>
       <geometry>
-        <mesh filename="package://justina_description/meshes/justina/arm/Gripper_Clean.dae"/>
+        <mesh filename="package://justina_description/meshes/justina/arm/Gripper_Clean.dae" scale="1 1 1"/>
       </geometry>
     </visual>
@@ -168,5 +168,5 @@
       <origin xyz="0 0 0" rpy="0 1.5707 0"/>
       <geometry>
-        <mesh filename="package://justina_description/meshes/justina/arm/Gripper_Clean.dae"/>
+        <mesh filename="package://justina_description/meshes/justina/arm/Gripper_Clean.dae" scale="1 1 1"/>
       </geometry>
     </collision>
@@ -174,6 +174,6 @@
   <!-- LEFT ARM JOINTS -->
   <joint name="left_torso_shoulder" type="revolute">
-    <origin xyz="0 0 0.01" rpy="0 0 0"/>
-    <parent link="shoulders_left_link"/>
+    <origin xyz="0 0 0.015" rpy="0 0 0"/>
+    <parent link="left_shoulder_link"/>
     <child link="left_shoulder_frame"/>
     <axis xyz="0 -1 0" />
@@ -182,5 +182,5 @@
   </joint>
   <joint name="left_shoulder_arm_motor" type="revolute">
-    <origin xyz="0 -0.009 -0.028" rpy="0 0 0"/>
+    <origin xyz="0 -0.009 -0.034" rpy="0 0 0"/>
     <parent link="left_shoulder_frame"/>
     <child link="left_arm"/>
@@ -198,5 +198,5 @@
   </joint>
   <joint name="left_wrist" type="revolute">
-    <origin xyz="0.009 0.001 -0.25" rpy="0 0 0"/>
+    <origin xyz="0.005 0.00 -0.25" rpy="0 0 0"/>
     <parent link="left_forearm"/>
     <child link="left_gripper_motors"/>
@@ -205,16 +205,16 @@
     <limit effort="16.0" velocity="3.0" lower="-1.7" upper="1.7"/>
   </joint>
-  <joint name="left_right_jaw_joint" type="revolute">
-    <origin xyz="0 -0.04 0" rpy="0 0 0"/>
+  <joint name="left_jaw_right_joint" type="revolute">
+    <origin xyz="0.002 -0.04 0" rpy="0 0 0"/>
     <parent link="left_gripper_motors"/>
-    <child link="left_right_jaw"/>
+    <child link="left_jaw_right"/>
     <axis xyz="-1 0 0" />
     <dynamics damping ="0.1" />
     <limit effort="16.0" velocity="3.0" lower="-1.7" upper="1.7"/>
   </joint>
-  <joint name="left_left_jaw_joint" type="revolute">
-    <origin xyz="0 0.04 0" rpy="0 0 0"/>
+  <joint name="left_jaw_left_joint" type="revolute">
+    <origin xyz="0.002 0.04 0" rpy="0 0 0"/>
     <parent link="left_gripper_motors"/>
-    <child link="left_left_jaw"/>
+    <child link="left_jaw_left"/>
     <axis xyz="-1 0 0" />
     <dynamics damping ="0.1" />
