Commit message: Virtual justina: edit mesh to match real robot dimensions, rename links and joints in both arms, add new colliders

File: urdf/justina_gazebo/justina_right_arm_low_poly.xacro (robot description, xacro)
@@ -1,8 +1,7 @@
 <?xml version="1.0"?>
-<robot name="justina_right_arm"
-  xmlns:xacro="http://www.ros.org/wiki/xacro">
+<robot name="justina_right_arm" xmlns:xacro="http://www.ros.org/wiki/xacro">
   <!--xacro:include filename="$(find justina_description)/urdf/justina/components/justina_right_arm.gazebo"/-->
   <!-- RIGHT ARM LINKS -->
-  <link name="shoulders_right_link">
+  <link name="right_shoulder_link">
     <inertial>
       <origin xyz="0 -0.01 0.02" rpy = "0 0 0"/>
@@ -13,5 +12,5 @@
       <origin xyz="0 -0.01 0.02" rpy = "0 3.1415 0"/>
       <geometry>
-        <mesh filename="package://justina_description/meshes/justina/servos/Servo_Mx106-2_LowPoly.dae"/>
+        <mesh filename="package://justina_description/meshes/justina/servos/Servo_Mx106-2_LowPoly.dae" scale="1 1 1"/>
       </geometry>
     </visual>
@@ -19,9 +18,9 @@
       <origin xyz="0 -0.01 0.02" rpy = "0 3.1415 0"/>
       <geometry>
-        <mesh filename="package://justina_description/meshes/justina/servos/Servo_Mx106-2_LowPoly.dae"/>
-      </geometry>
-    </collision>
-  </link>
-  <link name="shoulder_frame">
+        <mesh filename="package://justina_description/meshes/justina/servos/Servo_Mx106-2_LowPoly.dae" scale="1 1 1"/>
+      </geometry>
+    </collision>
+  </link>
+  <link name="right_shoulder_frame">
     <inertial>
       <origin xyz="0 -0.01 0.01" rpy = "0 0 -1.5707"/>
@@ -32,5 +31,5 @@
       <origin xyz="0 -0.01 0.01" rpy="0 0 -1.5707"/>
       <geometry>
-        <mesh filename="package://justina_description/meshes/justina/arm/Shoulder_Frame_LowPoly.dae"/>
+        <mesh filename="package://justina_description/meshes/justina/arm/Shoulder_Frame_LowPoly.dae" scale="1 1 1"/>
       </geometry>
     </visual>
@@ -38,9 +37,9 @@
       <origin xyz="0 -0.01 0.01" rpy="0 0 -1.5707"/>
       <geometry>
-        <mesh filename="package://justina_description/meshes/justina/arm/Shoulder_Frame_LowPoly.dae"/>
-      </geometry>
-    </collision>
-  </link>
-  <link name="arm">
+        <mesh filename="package://justina_description/meshes/justina/arm/Shoulder_Frame_LowPoly.dae" scale="1 1 1"/>
+      </geometry>
+    </collision>
+  </link>
+  <link name="right_arm">
     <inertial>
       <origin xyz="0 0 0" rpy = "0 0 0"/>
@@ -51,5 +50,5 @@
       <origin xyz="0 0 -0.02" rpy="0 0 3.1416"/>
       <geometry>
-        <mesh filename="package://justina_description/meshes/justina/servos/Servo_Mx64_LowPoly.dae"/>
+        <mesh filename="package://justina_description/meshes/justina/servos/Servo_Mx64_LowPoly.dae" scale="1 1 1"/>
       </geometry>
     </visual>
@@ -57,5 +56,5 @@
       <origin xyz="0 0 -0.02" rpy="0 0 3.1416"/>
       <geometry>
-        <mesh filename="package://justina_description/meshes/justina/servos/Servo_Mx64_LowPoly.dae"/>
+        <mesh filename="package://justina_description/meshes/justina/servos/Servo_Mx64_LowPoly.dae" scale="1 1 1"/>
       </geometry>
     </collision>
@@ -63,5 +62,5 @@
       <origin xyz="0 0 -0.216" rpy="0 3.1416 -1.5707"/>
       <geometry>
-        <mesh filename="package://justina_description/meshes/justina/arm/Arm_LowPoly.dae"/>
+        <mesh filename="package://justina_description/meshes/justina/arm/Arm_LowPoly.dae" scale="1 1 1"/>
       </geometry>
     </visual>
@@ -69,9 +68,9 @@
       <origin xyz="0 0 -0.216" rpy="0 3.1416 -1.5707"/>
       <geometry>
-        <mesh filename="package://justina_description/meshes/justina/arm/Arm_LowPoly.dae"/>
-      </geometry>
-    </collision>
-  </link>
-  <link name="forearm">
+        <mesh filename="package://justina_description/meshes/justina/arm/Arm_LowPoly.dae" scale="1 1 1"/>
+      </geometry>
+    </collision>
+  </link>
+  <link name="rigth_forearm">
     <inertial>
       <origin xyz="0 0 0" rpy = "0 0 0"/>
@@ -82,5 +81,5 @@
       <origin xyz="0 0 0" rpy="1.5707 0 0"/>
       <geometry>
-        <mesh filename="package://justina_description/meshes/justina/servos/Servo_Mx106_LowPoly.dae"/>
+        <mesh filename="package://justina_description/meshes/justina/servos/Servo_Mx106_LowPoly.dae" scale="1 1 1"/>
       </geometry>
     </visual>
@@ -88,5 +87,5 @@
       <origin xyz="0 0 0" rpy="1.5707 0 0"/>
       <geometry>
-        <mesh filename="package://justina_description/meshes/justina/servos/Servo_Mx106_LowPoly.dae"/>
+        <mesh filename="package://justina_description/meshes/justina/servos/Servo_Mx106_LowPoly.dae" scale="1 1 1"/>
       </geometry>
     </collision>
@@ -94,5 +93,5 @@
       <origin xyz="0 0 -0.12" rpy="0 0 1.5707"/>
       <geometry>
-        <mesh filename="package://justina_description/meshes/justina/arm/Forearm_LowPoly.dae"/>
+        <mesh filename="package://justina_description/meshes/justina/arm/Forearm_LowPoly.dae" scale="1 1 1"/>
       </geometry>
     </visual>
@@ -100,5 +99,5 @@
       <origin xyz="0 0 -0.12" rpy="0 0 1.5707"/>
       <geometry>
-        <mesh filename="package://justina_description/meshes/justina/arm/Forearm_LowPoly.dae"/>
+        <mesh filename="package://justina_description/meshes/justina/arm/Forearm_LowPoly.dae" scale="1 1 1"/>
       </geometry>
     </collision>
@@ -106,5 +105,5 @@
       <origin xyz="0.009 0.001 -0.21" rpy="0 0 -1.5707"/>
       <geometry>
-        <mesh filename="package://justina_description/meshes/justina/servos/Servo_Mx64_LowPoly.dae"/>
+        <mesh filename="package://justina_description/meshes/justina/servos/Servo_Mx64_LowPoly.dae" scale="1 1 1"/>
       </geometry>
     </visual>
@@ -112,9 +111,9 @@
       <origin xyz="0.009 0.001 -0.21" rpy="0 0 -1.5707"/>
       <geometry>
-        <mesh filename="package://justina_description/meshes/justina/servos/Servo_Mx64_LowPoly.dae"/>
-      </geometry>
-    </collision>
-  </link>
-  <link name="gripper_motors">
+        <mesh filename="package://justina_description/meshes/justina/servos/Servo_Mx64_LowPoly.dae" scale="1 1 1"/>
+      </geometry>
+    </collision>
+  </link>
+  <link name="right_gripper_motors">
     <inertial>
       <origin xyz="0 0 0" rpy = "0 0 0"/>
@@ -125,5 +124,5 @@
       <origin xyz="0 -0.004 0" rpy="1.5707 -1.5707 0"/>
       <geometry>
-        <mesh filename="package://justina_description/meshes/justina/servos/Servo_Mx28-2_LowPoly.dae"/>
+        <mesh filename="package://justina_description/meshes/justina/servos/Servo_Mx28-2_LowPoly.dae" scale="1 1 1"/>
       </geometry>
     </visual>
@@ -131,9 +130,9 @@
       <origin xyz="0 -0.004 0" rpy="1.5707 -1.5707 0"/>
       <geometry>
-        <mesh filename="package://justina_description/meshes/justina/servos/Servo_Mx28-2_LowPoly.dae"/>
-      </geometry>
-    </collision>
-  </link>
-  <link name="right_jaw">
+        <mesh filename="package://justina_description/meshes/justina/servos/Servo_Mx28-2_LowPoly.dae" scale="1 1 1"/>
+      </geometry>
+    </collision>
+  </link>
+  <link name="right_jaw_right">
     <inertial>
       <origin xyz="0 0 0" rpy = "0 0 0"/>
@@ -144,5 +143,5 @@
       <origin xyz="0 0 0" rpy="0 1.5707 3.1416"/>
       <geometry>
-        <mesh filename="package://justina_description/meshes/justina/arm/Gripper_Clean.dae"/>
+        <mesh filename="package://justina_description/meshes/justina/arm/Gripper_Clean.dae" scale="1 1 1"/>
       </geometry>
     </visual>
@@ -150,9 +149,9 @@
       <origin xyz="0 0 0" rpy="0 1.5707 3.1416"/>
       <geometry>
-        <mesh filename="package://justina_description/meshes/justina/arm/Gripper_Clean.dae"/>
-      </geometry>
-    </collision>
-  </link>
-  <link name="left_jaw">
+        <mesh filename="package://justina_description/meshes/justina/arm/Gripper_Clean.dae" scale="1 1 1"/>
+      </geometry>
+    </collision>
+  </link>
+  <link name="right_jaw_left">
     <inertial>
       <origin xyz="0 0 0" rpy = "0 0 0"/>
@@ -163,5 +162,5 @@
       <origin xyz="0 0 0" rpy="0 1.5707 0"/>
       <geometry>
-        <mesh filename="package://justina_description/meshes/justina/arm/Gripper_Clean.dae"/>
+        <mesh filename="package://justina_description/meshes/justina/arm/Gripper_Clean.dae" scale="1 1 1"/>
       </geometry>
     </visual>
@@ -169,5 +168,5 @@
       <origin xyz="0 0 0" rpy="0 1.5707 0"/>
       <geometry>
-        <mesh filename="package://justina_description/meshes/justina/arm/Gripper_Clean.dae"/>
+        <mesh filename="package://justina_description/meshes/justina/arm/Gripper_Clean.dae" scale="1 1 1"/>
       </geometry>
     </collision>
@@ -175,56 +174,51 @@
   <!-- <link name="right_arm_grip"/> -->
   <!-- RIGHT ARM JOINTS -->
-  <joint name="torso_shoulder" type="revolute">
+  <joint name="right_torso_shoulder" type="revolute">
     <origin xyz="0 0 0.01" rpy="0 0 0"/>
-    <parent link="shoulders_right_link"/>
-    <child link="shoulder_frame"/>
+    <parent link="right_shoulder_link"/>
+    <child link="right_shoulder_frame"/>
     <axis xyz="0 -1 0" />
     <dynamics damping ="0.1" />
     <limit effort="16.0" velocity="3.0" lower="-1.7" upper="1.7"/>
   </joint>
-  <joint name="shoulder_arm_motor" type="revolute">
+  <joint name="right_shoulder_arm_motor" type="revolute">
     <origin xyz="0 -0.009 -0.028" rpy="0 0 0"/>
-    <parent link="shoulder_frame"/>
-    <child link="arm"/>
+    <parent link="right_shoulder_frame"/>
+    <child link="right_arm"/>
     <axis xyz="0 0 -1" />
     <dynamics damping ="0.1" />
     <limit effort="16.0" velocity="3.0" lower="-1.7" upper="1.7"/>
   </joint>
-  <joint name="elbow" type="revolute">
+  <joint name="right_elbow" type="revolute">
     <origin xyz="0 0.002 -0.216" rpy="0 0 0"/>
-    <parent link="arm"/>
-    <child link="forearm"/>
+    <parent link="right_arm"/>
+    <child link="rigth_forearm"/>
     <axis xyz="0 -1 0" />
     <dynamics damping ="0.1" />
     <limit effort="16.0" velocity="3.0" lower="-1.7" upper="1.7"/>
   </joint>
-  <joint name="wrist" type="revolute">
+  <joint name="right_wrist" type="revolute">
     <origin xyz="0.009 0.001 -0.25" rpy="0 0 0"/>
-    <parent link="forearm"/>
-    <child link="gripper_motors"/>
+    <parent link="rigth_forearm"/>
+    <child link="right_gripper_motors"/>
     <axis xyz="0 0 -1" />
     <dynamics damping ="0.1" />
     <limit effort="16.0" velocity="3.0" lower="-1.7" upper="1.7"/>
   </joint>
-  <joint name="right_jaw_joint" type="revolute">
+  <joint name="right_jaw_right_joint" type="revolute">
     <origin xyz="0 -0.04 0" rpy="0 0 0"/>
-    <parent link="gripper_motors"/>
-    <child link="right_jaw"/>
+    <parent link="right_gripper_motors"/>
+    <child link="right_jaw_right"/>
     <axis xyz="-1 0 0" />
     <dynamics damping ="0.1" />
     <limit effort="16.0" velocity="3.0" lower="-1.7" upper="1.7"/>
   </joint>
-  <joint name="left_jaw_joint" type="revolute">
+  <joint name="right_jaw_left_joint" type="revolute">
     <origin xyz="0 0.04 0" rpy="0 0 0"/>
-    <parent link="gripper_motors"/>
-    <child link="left_jaw"/>
+    <parent link="right_gripper_motors"/>
+    <child link="right_jaw_left"/>
     <axis xyz="-1 0 0" />
     <dynamics damping ="0.1" />
     <limit effort="16.0" velocity="3.0" lower="-1.7" upper="1.7"/>
   </joint>
-  <!-- <joint name="right_grip_center_joint" type="fixed">
-    <origin xyz="0 0 -0.12" rpy="0 0 0"/>
-    <parent link="gripper_motors"/>
-    <child link="right_arm_grip"/>
-  </joint> -->
 </robot>

File: urdf/justina_gazebo/justina_toso_low_poly.xacro (robot description, xacro)
@@ -10,17 +10,17 @@
         <inertial>
             <mass value="${torso_mass}"/>
-            <origin xyz= "0 0 -0.55" rpy="0 0 0"/>
+            <origin xyz= "0 0 -0.1" rpy="0 0 0"/>
             <xacro:box_inertia m="${torso_mass}" x="0.07" y="0.09" z="0.05"/>
         </inertial>
         <visual>
-            <origin xyz= "0.0 0.0 -0.1" rpy="0 0 0"/>
+            <origin xyz= "0.0 0.0 0.0" rpy="0 0 0"/>
             <geometry>
-                <mesh filename="package://justina_description/meshes/justina/torso/Justina_Torso_LowPoly.dae"/>
+                <mesh filename="package://justina_description/meshes/justina/torso/Justina_Torso_LowPoly.dae" scale="1 1 1"/>
             </geometry>
         </visual>
         <collision>
-            <origin xyz= "0.0 0.0 -0.1" rpy="0 0 0"/>
+            <origin xyz= "0.0 0.0 0.0" rpy="0 0 0"/>
             <geometry>
-                <mesh filename="package://justina_description/meshes/justina/torso/Justina_Torso_LowPoly.dae"/>
+                <mesh filename="package://justina_description/meshes/justina/torso/Justina_Torso_LowPoly.dae" scale="1 1 1"/>
             </geometry>
         </collision>
@@ -28,5 +28,5 @@
     <joint name="spine_connect" type="fixed">
         <origin xyz= "0.0 0 0.35" rpy="0 0 0"/>
-        <parent link="torso_link"/>
+        <parent link="torso_link"/>5
         <child link="spine_link"/>
     </joint>
