Commit message: Create clean URF from blender, fix mesh and link-joint issues

File: urdf/justina_gazebo/festina_base_low_poly.xacro (robot description, xacro)
@@ -37,7 +37,7 @@
             </visual>
             <collision>
-                <origin xyz="0 0 0" rpy="1.570796 0 0"/>
+                <origin xyz="0 0 0" rpy="0 0 0"/>
                 <geometry>
-                    <cylinder radius="0.062" length="0.058"/>
+                    <mesh filename="package://justina_description/meshes/robotino_low_poly/Robotino3_SplitWheel_Collider.dae" scale="1 1 1"/>
                 </geometry>
             </collision>
@@ -72,5 +72,5 @@
         </inertial>
         <visual>
-            <origin xyz="0 0 0" rpy="0 0 1.57"/>
+            <origin xyz="0 0 0" rpy="0 0 0"/>
             <geometry>
                 <mesh filename="package://justina_description/meshes/robotino_low_poly/sensors/Hokuyo_Clean.dae" scale="1 1 1"/>

File: urdf/justina_gazebo/justina_head_low_poly.xacro (robot description, xacro)
@@ -11,5 +11,5 @@
     </inertial>
     <visual>
-      <origin xyz= "0.0 0 0.01" rpy="0 0 -${M_PI/2}"/>
+      <origin xyz= "0.0 0 0.01" rpy="0 0 0"/>
       <geometry>
         <mesh filename="package://justina_description/meshes/justina/servos/Servo_Mx64_LowPoly.dae" scale="1 1 1"/>
@@ -17,5 +17,5 @@
     </visual>
     <collision>
-      <origin xyz= "0.0 0 0.01" rpy="0 0 -${M_PI/2}"/>
+      <origin xyz= "0.0 0 0.01" rpy="0 0 0"/>
       <geometry>
         <mesh filename="package://justina_description/meshes/justina/servos/Servo_Mx64_LowPoly.dae" scale="1 1 1"/>
@@ -30,5 +30,5 @@
     </inertial>
     <visual>
-      <origin xyz= "0 0.0 0.06" rpy="${M_PI/2} 0 0"/>
+      <origin xyz= "0 0.0 0.06" rpy="${M_PI/2} -${M_PI/2} 0"/>
       <geometry>
         <mesh filename="package://justina_description/meshes/justina/servos/Servo_Mx64_LowPoly.dae" scale="1 1 1"/>
@@ -36,5 +36,5 @@
     </visual>
     <collision>
-      <origin xyz= "0 0.0 0.06" rpy="${M_PI/2} 0 0"/>
+      <origin xyz= "0 0.0 0.06" rpy="${M_PI/2} -${M_PI/2} 0"/>
       <geometry>
         <mesh filename="package://justina_description/meshes/justina/servos/Servo_Mx64_LowPoly.dae" scale="1 1 1"/>

File: urdf/justina_gazebo/justina_left_arm_low_poly.xacro (robot description, xacro)
@@ -10,5 +10,5 @@
     </inertial>
     <visual>
-      <origin xyz="0 -0.01 0.02" rpy = "0 3.1415 0"/>
+      <origin xyz="0 -0.01 0.02" rpy = "0 0 0"/>
       <geometry>
         <mesh filename="package://justina_description/meshes/justina/servos/Servo_Mx106-2_LowPoly.dae" scale="1 1 1"/>
@@ -16,5 +16,5 @@
     </visual>
     <collision>
-      <origin xyz="0 -0.01 0.02" rpy = "0 3.1415 0"/>
+      <origin xyz="0 -0.01 0.02" rpy = "0 0 0"/>
       <geometry>
         <mesh filename="package://justina_description/meshes/justina/servos/Servo_Mx106-2_LowPoly.dae" scale="1 1 1"/>
@@ -24,10 +24,10 @@
   <link name="left_shoulder_frame">
     <inertial>
-      <origin xyz="0 -0.01 0.0" rpy = "0 0 -1.5707"/>
+      <origin xyz="0 -0.01 0.0" rpy = "0 0 0"/>
       <mass value="0.08146"/>
       <inertia ixx="0.0000813217" ixy="0.0" ixz="0.0" iyy="0.000196" iyz="0.0" izz="0.0001282"/>
     </inertial>
     <visual>
-      <origin xyz="0 -0.01 0.0" rpy="0 0 -1.5707"/>
+      <origin xyz="0 -0.01 0.0" rpy="0 0 0"/>
       <geometry>
         <mesh filename="package://justina_description/meshes/justina/arm/Shoulder_Frame_LowPoly.dae" scale="1 1 1"/>
@@ -35,5 +35,5 @@
     </visual>
     <collision>
-      <origin xyz="0 -0.01 0.0" rpy="0 0 -1.5707"/>
+      <origin xyz="0 -0.01 0.0" rpy="0 0 0"/>
       <geometry>
         <mesh filename="package://justina_description/meshes/justina/arm/Shoulder_Frame_LowPoly.dae" scale="1 1 1"/>
@@ -48,17 +48,17 @@
     </inertial>
     <visual>
-      <origin xyz="0 0 -0.02" rpy="0 0 6.2822"/>
-      <geometry>
-        <mesh filename="package://justina_description/meshes/justina/servos/Servo_Mx64_LowPoly.dae" scale="1 1 1"/>
-      </geometry>
-    </visual>
-    <collision>
-      <origin xyz="0 0 -0.02" rpy="0 0 6.2822"/>
-      <geometry>
-        <mesh filename="package://justina_description/meshes/justina/servos/Servo_Mx64_LowPoly.dae" scale="1 1 1"/>
-      </geometry>
-    </collision>
-    <visual>
-      <origin xyz="0 0 -0.216" rpy="0 3.1416 1.5707"/>
+      <origin xyz="0 0 -0.02" rpy="0 0 1.5707"/>
+      <geometry>
+        <mesh filename="package://justina_description/meshes/justina/servos/Servo_Mx64_LowPoly.dae" scale="1 1 1"/>
+      </geometry>
+    </visual>
+    <collision>
+      <origin xyz="0 0 -0.02" rpy="0 0 1.5707"/>
+      <geometry>
+        <mesh filename="package://justina_description/meshes/justina/servos/Servo_Mx64_LowPoly.dae" scale="1 1 1"/>
+      </geometry>
+    </collision>
+    <visual>
+      <origin xyz="0 0 -0.216" rpy="0 0 1.5707"/>
       <geometry>
         <mesh filename="package://justina_description/meshes/justina/arm/Arm_LowPoly.dae" scale="1 1 1"/>
@@ -66,5 +66,5 @@
     </visual>
     <collision>
-      <origin xyz="0 0 -0.216" rpy="0 3.1416 1.5707"/>
+      <origin xyz="0 0 -0.216" rpy="0 0 1.5707"/>
       <geometry>
         <mesh filename="package://justina_description/meshes/justina/arm/Arm_LowPoly.dae" scale="1 1 1"/>
@@ -79,5 +79,5 @@
     </inertial>
     <visual>
-      <origin xyz="0 0 0" rpy="1.5707 0 0"/>
+      <origin xyz="0 0 0" rpy="0 0 0"/>
       <geometry>
         <mesh filename="package://justina_description/meshes/justina/servos/Servo_Mx106_LowPoly.dae" scale="1 1 1"/>
@@ -85,5 +85,5 @@
     </visual>
     <collision>
-      <origin xyz="0 0 0" rpy="1.5707 0 0"/>
+      <origin xyz="0 0 0" rpy="0 0 0"/>
       <geometry>
         <mesh filename="package://justina_description/meshes/justina/servos/Servo_Mx106_LowPoly.dae" scale="1 1 1"/>
@@ -91,5 +91,5 @@
     </collision>
     <visual>
-      <origin xyz="0 0 -0.12" rpy="0 0 1.5707"/>
+      <origin xyz="0 0 -0.12" rpy="0 0 0"/>
       <geometry>
         <mesh filename="package://justina_description/meshes/justina/arm/Forearm_LowPoly.dae" scale="1 1 1"/>
@@ -97,5 +97,5 @@
     </visual>
     <collision>
-      <origin xyz="0 0 -0.12" rpy="0 0 1.5707"/>
+      <origin xyz="0 0 -0.12" rpy="0 0 0"/>
       <geometry>
         <mesh filename="package://justina_description/meshes/justina/arm/Forearm_LowPoly.dae" scale="1 1 1"/>
@@ -103,11 +103,11 @@
     </collision>
     <visual>
-      <origin xyz="0.009 0.001 -0.21" rpy="0 0 -1.5707"/>
-      <geometry>
-        <mesh filename="package://justina_description/meshes/justina/servos/Servo_Mx64_LowPoly.dae" scale="1 1 1"/>
-      </geometry>
-    </visual>
-    <collision>
-      <origin xyz="0.009 0.001 -0.21" rpy="0 0 -1.5707"/>
+      <origin xyz="0.009 0.001 -0.21" rpy="0 0 0"/>
+      <geometry>
+        <mesh filename="package://justina_description/meshes/justina/servos/Servo_Mx64_LowPoly.dae" scale="1 1 1"/>
+      </geometry>
+    </visual>
+    <collision>
+      <origin xyz="0.009 0.001 -0.21" rpy="0 0 0"/>
       <geometry>
         <mesh filename="package://justina_description/meshes/justina/servos/Servo_Mx64_LowPoly.dae" scale="1 1 1"/>
@@ -122,5 +122,5 @@
     </inertial>
     <visual>
-      <origin xyz="0 0 0" rpy="1.5707 -1.5707 0"/>
+      <origin xyz="0 0 0" rpy="0 0 0"/>
       <geometry>
         <mesh filename="package://justina_description/meshes/justina/servos/Servo_Mx28-2_LowPoly.dae" scale="1 1 1"/>
@@ -128,5 +128,5 @@
     </visual>
     <collision>
-      <origin xyz="0 0 0" rpy="1.5707 -1.5707 0"/>
+      <origin xyz="0 0 0" rpy="0 0 0"/>
       <geometry>
         <mesh filename="package://justina_description/meshes/justina/servos/Servo_Mx28-2_LowPoly.dae" scale="1 1 1"/>
@@ -141,11 +141,11 @@
     </inertial>
     <visual>
-      <origin xyz="0 0 0" rpy="0 1.5707 3.1416"/>
-      <geometry>
-        <mesh filename="package://justina_description/meshes/justina/arm/Gripper_Clean.dae" scale="1 1 1"/>
-      </geometry>
-    </visual>
-    <collision>
-      <origin xyz="0 0 0" rpy="0 1.5707 3.1416"/>
+      <origin xyz="0 0 0" rpy="0 0 -1.5708"/>
+      <geometry>
+        <mesh filename="package://justina_description/meshes/justina/arm/Gripper_Clean.dae" scale="1 1 1"/>
+      </geometry>
+    </visual>
+    <collision>
+      <origin xyz="0 0 0" rpy="0 0 -1.5708"/>
       <geometry>
         <mesh filename="package://justina_description/meshes/justina/arm/Gripper_Clean.dae" scale="1 1 1"/>
@@ -160,11 +160,11 @@
     </inertial>
     <visual>
-      <origin xyz="0 0 0" rpy="0 1.5707 0"/>
-      <geometry>
-        <mesh filename="package://justina_description/meshes/justina/arm/Gripper_Clean.dae" scale="1 1 1"/>
-      </geometry>
-    </visual>
-    <collision>
-      <origin xyz="0 0 0" rpy="0 1.5707 0"/>
+      <origin xyz="0 0 0" rpy="0 0 1.5708"/>
+      <geometry>
+        <mesh filename="package://justina_description/meshes/justina/arm/Gripper_Clean.dae" scale="1 1 1"/>
+      </geometry>
+    </visual>
+    <collision>
+      <origin xyz="0 0 0" rpy="0 0 1.5708"/>
       <geometry>
         <mesh filename="package://justina_description/meshes/justina/arm/Gripper_Clean.dae" scale="1 1 1"/>
@@ -198,5 +198,5 @@
   </joint>
   <joint name="left_wrist" type="revolute">
-    <origin xyz="0.005 0.00 -0.25" rpy="0 0 0"/>
+    <origin xyz="0. 0.0 -0.25" rpy="0 0 0"/>
     <parent link="left_forearm"/>
     <child link="left_gripper_motors"/>

File: urdf/justina_gazebo/justina_right_arm_low_poly.xacro (robot description, xacro)
@@ -10,5 +10,5 @@
     </inertial>
     <visual>
-      <origin xyz="0 -0.01 0.02" rpy = "0 3.1415 0"/>
+      <origin xyz="0 -0.01 0.02" rpy = "0 0 0"/>
       <geometry>
         <mesh filename="package://justina_description/meshes/justina/servos/Servo_Mx106-2_LowPoly.dae" scale="1 1 1"/>
@@ -16,5 +16,5 @@
     </visual>
     <collision>
-      <origin xyz="0 -0.01 0.02" rpy = "0 3.1415 0"/>
+      <origin xyz="0 -0.01 0.02" rpy = "0 0 0"/>
       <geometry>
         <mesh filename="package://justina_description/meshes/justina/servos/Servo_Mx106-2_LowPoly.dae" scale="1 1 1"/>
@@ -29,5 +29,5 @@
     </inertial>
     <visual>
-      <origin xyz="0 -0.01 0.01" rpy="0 0 -1.5707"/>
+      <origin xyz="0 -0.01 0.0" rpy="0 0 0"/>
       <geometry>
         <mesh filename="package://justina_description/meshes/justina/arm/Shoulder_Frame_LowPoly.dae" scale="1 1 1"/>
@@ -35,5 +35,5 @@
     </visual>
     <collision>
-      <origin xyz="0 -0.01 0.01" rpy="0 0 -1.5707"/>
+      <origin xyz="0 -0.01 0.0" rpy="0 0 0"/>
       <geometry>
         <mesh filename="package://justina_description/meshes/justina/arm/Shoulder_Frame_LowPoly.dae" scale="1 1 1"/>
@@ -48,17 +48,17 @@
     </inertial>
     <visual>
-      <origin xyz="0 0 -0.02" rpy="0 0 3.1416"/>
-      <geometry>
-        <mesh filename="package://justina_description/meshes/justina/servos/Servo_Mx64_LowPoly.dae" scale="1 1 1"/>
-      </geometry>
-    </visual>
-    <collision>
-      <origin xyz="0 0 -0.02" rpy="0 0 3.1416"/>
-      <geometry>
-        <mesh filename="package://justina_description/meshes/justina/servos/Servo_Mx64_LowPoly.dae" scale="1 1 1"/>
-      </geometry>
-    </collision>
-    <visual>
-      <origin xyz="0 0 -0.216" rpy="0 3.1416 -1.5707"/>
+      <origin xyz="0 0 -0.02" rpy="0 0 -1.5707"/>
+      <geometry>
+        <mesh filename="package://justina_description/meshes/justina/servos/Servo_Mx64_LowPoly.dae" scale="1 1 1"/>
+      </geometry>
+    </visual>
+    <collision>
+      <origin xyz="0 0 -0.02" rpy="0 0 -1.5707"/>
+      <geometry>
+        <mesh filename="package://justina_description/meshes/justina/servos/Servo_Mx64_LowPoly.dae" scale="1 1 1"/>
+      </geometry>
+    </collision>
+    <visual>
+      <origin xyz="0 0 -0.216" rpy="0 0 -1.5707"/>
       <geometry>
         <mesh filename="package://justina_description/meshes/justina/arm/Arm_LowPoly.dae" scale="1 1 1"/>
@@ -66,5 +66,5 @@
     </visual>
     <collision>
-      <origin xyz="0 0 -0.216" rpy="0 3.1416 -1.5707"/>
+      <origin xyz="0 0 -0.216" rpy="0 0 -1.5707"/>
       <geometry>
         <mesh filename="package://justina_description/meshes/justina/arm/Arm_LowPoly.dae" scale="1 1 1"/>
@@ -79,5 +79,5 @@
     </inertial>
     <visual>
-      <origin xyz="0 0 0" rpy="1.5707 0 0"/>
+      <origin xyz="0 0 0" rpy="0 0 0"/>
       <geometry>
         <mesh filename="package://justina_description/meshes/justina/servos/Servo_Mx106_LowPoly.dae" scale="1 1 1"/>
@@ -85,5 +85,5 @@
     </visual>
     <collision>
-      <origin xyz="0 0 0" rpy="1.5707 0 0"/>
+      <origin xyz="0 0 0" rpy="0 0 0"/>
       <geometry>
         <mesh filename="package://justina_description/meshes/justina/servos/Servo_Mx106_LowPoly.dae" scale="1 1 1"/>
@@ -91,23 +91,23 @@
     </collision>
     <visual>
+      <origin xyz="0 0 -0.12" rpy="0 0 0"/>
+      <geometry>
+        <mesh filename="package://justina_description/meshes/justina/arm/Forearm_LowPoly.dae" scale="1 1 1"/>
+      </geometry>
+    </visual>
+    <collision>
       <origin xyz="0 0 -0.12" rpy="0 0 1.5707"/>
       <geometry>
         <mesh filename="package://justina_description/meshes/justina/arm/Forearm_LowPoly.dae" scale="1 1 1"/>
       </geometry>
-    </visual>
-    <collision>
-      <origin xyz="0 0 -0.12" rpy="0 0 1.5707"/>
-      <geometry>
-        <mesh filename="package://justina_description/meshes/justina/arm/Forearm_LowPoly.dae" scale="1 1 1"/>
-      </geometry>
-    </collision>
-    <visual>
-      <origin xyz="0.009 0.001 -0.21" rpy="0 0 -1.5707"/>
-      <geometry>
-        <mesh filename="package://justina_description/meshes/justina/servos/Servo_Mx64_LowPoly.dae" scale="1 1 1"/>
-      </geometry>
-    </visual>
-    <collision>
-      <origin xyz="0.009 0.001 -0.21" rpy="0 0 -1.5707"/>
+    </collision>
+    <visual>
+      <origin xyz="0.009 0.001 -0.21" rpy="0 0 0"/>
+      <geometry>
+        <mesh filename="package://justina_description/meshes/justina/servos/Servo_Mx64_LowPoly.dae" scale="1 1 1"/>
+      </geometry>
+    </visual>
+    <collision>
+      <origin xyz="0.009 0.001 -0.21" rpy="0 0 0"/>
       <geometry>
         <mesh filename="package://justina_description/meshes/justina/servos/Servo_Mx64_LowPoly.dae" scale="1 1 1"/>
@@ -122,5 +122,5 @@
     </inertial>
     <visual>
-      <origin xyz="0 -0.004 0" rpy="1.5707 -1.5707 0"/>
+      <origin xyz="0 -0.004 0" rpy="0 0 0"/>
       <geometry>
         <mesh filename="package://justina_description/meshes/justina/servos/Servo_Mx28-2_LowPoly.dae" scale="1 1 1"/>
@@ -128,5 +128,5 @@
     </visual>
     <collision>
-      <origin xyz="0 -0.004 0" rpy="1.5707 -1.5707 0"/>
+      <origin xyz="0 -0.004 0" rpy="0 0 0"/>
       <geometry>
         <mesh filename="package://justina_description/meshes/justina/servos/Servo_Mx28-2_LowPoly.dae" scale="1 1 1"/>
@@ -141,11 +141,11 @@
     </inertial>
     <visual>
-      <origin xyz="0 0 0" rpy="0 1.5707 3.1416"/>
-      <geometry>
-        <mesh filename="package://justina_description/meshes/justina/arm/Gripper_Clean.dae" scale="1 1 1"/>
-      </geometry>
-    </visual>
-    <collision>
-      <origin xyz="0 0 0" rpy="0 1.5707 3.1416"/>
+      <origin xyz="0 0 0" rpy="0 0 -1.5708"/>
+      <geometry>
+        <mesh filename="package://justina_description/meshes/justina/arm/Gripper_Clean.dae" scale="1 1 1"/>
+      </geometry>
+    </visual>
+    <collision>
+      <origin xyz="0 0 0" rpy="0 0 -1.5708"/>
       <geometry>
         <mesh filename="package://justina_description/meshes/justina/arm/Gripper_Clean.dae" scale="1 1 1"/>
@@ -160,11 +160,11 @@
     </inertial>
     <visual>
-      <origin xyz="0 0 0" rpy="0 1.5707 0"/>
-      <geometry>
-        <mesh filename="package://justina_description/meshes/justina/arm/Gripper_Clean.dae" scale="1 1 1"/>
-      </geometry>
-    </visual>
-    <collision>
-      <origin xyz="0 0 0" rpy="0 1.5707 0"/>
+      <origin xyz="0 0 0" rpy="0 0 1.5708"/>
+      <geometry>
+        <mesh filename="package://justina_description/meshes/justina/arm/Gripper_Clean.dae" scale="1 1 1"/>
+      </geometry>
+    </visual>
+    <collision>
+      <origin xyz="0 0 0" rpy="0 0 1.5708"/>
       <geometry>
         <mesh filename="package://justina_description/meshes/justina/arm/Gripper_Clean.dae" scale="1 1 1"/>
@@ -175,5 +175,5 @@
   <!-- RIGHT ARM JOINTS -->
   <joint name="right_torso_shoulder" type="revolute">
-    <origin xyz="0 0 0.01" rpy="0 0 0"/>
+    <origin xyz="0 0 0.015" rpy="0 0 0"/>
     <parent link="right_shoulder_link"/>
     <child link="right_shoulder_frame"/>
@@ -183,5 +183,5 @@
   </joint>
   <joint name="right_shoulder_arm_motor" type="revolute">
-    <origin xyz="0 -0.009 -0.028" rpy="0 0 0"/>
+    <origin xyz="0 -0.009 -0.038" rpy="0 0 0"/>
     <parent link="right_shoulder_frame"/>
     <child link="right_arm"/>
