Commit message: Fix URDF positions in torso and grippers, set physics materials in wbt, add teleoperate controller

File: webots_env/urdf/Robot.urdf (robot description, URDF)
Before this commit: robot justina, 32 links, 31 joints
Links:
- removed link kinect_color_frame
- removed link kinect_depth_frame
- added link base_footprint
- added link camera_color_frame
- added link camera_color_optical_frame
- added link camera_depth_frame
- added link camera_depth_optical_frame
Joints:
- removed joint camera_to_color
- removed joint camera_to_depth
- added joint base_footprint_joint: type fixed, parent base_footprint, child base_link, origin xyz=0 0 0.06 rpy=0 0 0
- added joint camera_color_joint: type fixed, parent camera_link, child camera_color_frame, origin xyz=0 0 0 rpy=0 0 0
- added joint camera_color_optical_joint: type fixed, parent camera_color_frame, child camera_color_optical_frame, origin xyz=0 0 0 rpy=-1.5708 0 -1.5708
- added joint camera_depth_joint: type fixed, parent camera_link, child camera_depth_frame, origin xyz=0 0 0 rpy=0 0 0
- added joint camera_depth_optical_joint: type fixed, parent camera_depth_frame, child camera_depth_optical_frame, origin xyz=0 0 0 rpy=-1.5708 0 -1.5708
- joint left_griper_L_joint: origin xyz=0 0.01614 -0.169349 rpy=0 0 0 -> xyz=0 0.01614 -0.169349 rpy=0 0 -1.5708
- joint left_griper_R_joint: origin xyz=0 -0.01614 -0.169349 rpy=0 0 0 -> xyz=0 -0.01614 -0.169349 rpy=0 0 1.5708
- joint right_griper_L_joint: origin xyz=0 0.01614 -0.169349 rpy=0 0 0 -> xyz=0 0.01614 -0.169349 rpy=0 0 -1.5708
- joint right_griper_R_joint: origin xyz=0 -0.01614 -0.169349 rpy=0 0 0 -> xyz=0 -0.01614 -0.169349 rpy=0 0 1.5708
- joint torso_joint: origin xyz=0 0 0 rpy=0 0 0 -> xyz=0 0 0.08 rpy=0 0 0
- joint wheel0_joint: origin xyz=-0.165 0 0.063899 rpy=0 0 1.5708 -> xyz=-0.18 0 0.06 rpy=0 0 1.5708
- joint wheel1_joint: origin xyz=0.0825 -0.142894 0.063899 rpy=0 0 -2.61799 -> xyz=0.09 -0.155885 0.06 rpy=0 0 -2.61799
- joint wheel2_joint: origin xyz=0.0825 0.142894 0.063899 rpy=0 0 -0.5236 -> xyz=0.09 0.155885 0.06 rpy=0 0 -0.523599

Commit message: Fix wheel link names and update virtual topic names to match real ones

File: webots_env/urdf/Robot.urdf (robot description, URDF)
Before this commit: robot justina, 35 links, 34 joints
Joints:
- joint base_footprint_joint: origin xyz=0 0 0.06 rpy=0 0 0 -> xyz=0 0 0 rpy=0 0 0
- joint wheel0_joint: origin xyz=-0.18 0 0.06 rpy=0 0 1.5708 -> xyz=0.09 0.155885 0.06 rpy=0 0 -0.523599
- joint wheel1_joint: origin xyz=0.09 -0.155885 0.06 rpy=0 0 -2.61799 -> xyz=-0.18 0 0.06 rpy=0 0 1.5708
- joint wheel2_joint: origin xyz=0.09 0.155885 0.06 rpy=0 0 -0.523599 -> xyz=0.09 -0.155885 0.06 rpy=0 0 -2.61799

Commit message: Fix joint rotation axis from arms in wbt, add hokuyo mesh in URDF and fix wheels rotation axis

File: webots_env/urdf/Robot.urdf (robot description, URDF)
Before this commit: robot justina, 35 links, 34 joints
Links:
- link laser_link: geometry collision box size=0.05 0.05455 0.07; visual mesh filename=package://justina_description/meshes/robotino_low_poly/sens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
Joints:
- joint wheel0_joint: axis 0 1 0 -> 0 -1 0
- joint wheel1_joint: axis 0 1 0 -> 0 -1 0
- joint wheel2_joint: axis 0 1 0 -> 0 -1 0

Commit message: Deleted all unused meshes and updated justina.urdf

File: webots_env/urdf/Robot.urdf (robot description, URDF)
Before this commit: robot justina, 35 links, 34 joints
Links:
- link base_link: geometry collision mesh filename=package://justina_description/meshes/justina/Base_Collider_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; visual mesh filename=package://justina_description/meshes/justina/Base_ROBOTINO_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
- link body_link: geometry collision mesh filename=package://justina_description/meshes/justina/Body_Collider_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; visual mesh filename=package://justina_description/meshes/justina/Body_ROBOTINO_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
- link camera_link: geometry collision mesh filename=package://justina_description/meshes/justina/face/SingleKin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; visual mesh filename=package://justina_description/meshes/justina/face/SingleKin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
- link head_frame_link: geometry collision mesh filename=package://justina_description/meshes/justina/face/Face_Fram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; visual mesh filename=package://justina_description/meshes/justina/face/Face_Fram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
- link head_link: geometry collision mesh filename=package://justina_description/meshes/justina/face/HeadTiltM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; visual mesh filename=package://justina_description/meshes/justina/face/HeadTiltM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
- link l_arm_link: geometry collision mesh filename=package://justina_description/meshes/justina/arm/Arm_Collid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; visual mesh filename=package://justina_description/meshes/justina/arm/Arm.dae
- link l_arm_twist_link: geometry collision mesh filename=package://justina_description/meshes/justina/arm/ArmTwist_C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; visual mesh filename=package://justina_description/meshes/justina/arm/ArmTwist.d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
- link l_forearm_link: geometry collision mesh filename=package://justina_description/meshes/justina/arm/Forearm_Co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; visual mesh filename=package://justina_description/meshes/justina/arm/Forearm.dae
- link l_hand_link: geometry collision mesh filename=package://justina_description/meshes/justina/arm/Gripper_Ha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; visual mesh filename=package://justina_description/meshes/justina/arm/Gripper_Ha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
- link l_wrist_link: geometry collision mesh filename=package://justina_description/meshes/justina/arm/Wrist_Coll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; visual mesh filename=package://justina_description/meshes/justina/arm/Wrist.dae
- link laser_link: geometry collision box size=0.05 0.05455 0.07; visual mesh filename=package://justina_description/meshes/robotino/sensors/Hokuy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
- link left_griper_L_link: geometry collision mesh filename=package://justina_description/meshes/justina/arm/Gripper_Co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; visual mesh filename=package://justina_description/meshes/justina/arm/Gripper.dae
- link left_griper_R_link: geometry collision mesh filename=package://justina_description/meshes/justina/arm/Gripper_Co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; visual mesh filename=package://justina_description/meshes/justina/arm/Gripper.dae
- link left_shoulder_link: geometry collision mesh filename=package://justina_description/meshes/justina/arm/ShoulderMo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; visual mesh filename=package://justina_description/meshes/justina/arm/ShoulderMo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
- link lf_frame_link: geometry collision mesh filename=package://justina_description/meshes/justina/arm/ShoulderFr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; visual mesh filename=package://justina_description/meshes/justina/arm/ShoulderFr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
- link neck_link: geometry collision mesh filename=package://justina_description/meshes/justina/Neck_Collider.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; visual mesh filename=package://justina_description/meshes/justina/Neck.dae
- link r_arm_link: geometry collision mesh filename=package://justina_description/meshes/justina/arm/Arm_Collid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; visual mesh filename=package://justina_description/meshes/justina/arm/Arm.dae
- link r_arm_twist_link: geometry collision mesh filename=package://justina_description/meshes/justina/arm/ArmTwist_C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; visual mesh filename=package://justina_description/meshes/justina/arm/ArmTwist.d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
- link r_forearm_link: geometry collision mesh filename=package://justina_description/meshes/justina/arm/Forearm_Co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; visual mesh filename=package://justina_description/meshes/justina/arm/Forearm.dae
- link r_hand_link: geometry collision mesh filename=package://justina_description/meshes/justina/arm/Gripper_Ha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; visual mesh filename=package://justina_description/meshes/justina/arm/Gripper_Ha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
- link r_wrist_link: geometry collision mesh filename=package://justina_description/meshes/justina/arm/Wrist_Coll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; visual mesh filename=package://justina_description/meshes/justina/arm/Wrist.dae
- link rf_frame_link: geometry collision mesh filename=package://justina_description/meshes/justina/arm/ShoulderFr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; visual mesh filename=package://justina_description/meshes/justina/arm/ShoulderFr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
- link right_griper_L_link: geometry collision mesh filename=package://justina_description/meshes/justina/arm/Gripper_Co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; visual mesh filename=package://justina_description/meshes/justina/arm/Gripper.dae
- link right_griper_R_link: geometry collision mesh filename=package://justina_description/meshes/justina/arm/Gripper_Co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; visual mesh filename=package://justina_description/meshes/justina/arm/Gripper.dae
- link right_shoulder_link: geometry collision mesh filename=package://justina_description/meshes/justina/arm/ShoulderMo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; visual mesh filename=package://justina_description/meshes/justina/arm/ShoulderMo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
- link spine_link: geometry collision mesh filename=package://justina_description/meshes/justina/ShoulderPads.d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; visual mesh filename=package://justina_description/meshes/justina/ShoulderPads.d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
- link torso_link: geometry collision mesh filename=package://justina_description/meshes/justina/Torso_Collider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; visual mesh filename=package://justina_description/meshes/justina/Torso_ROBOTINO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
- link wheel0_link: geometry collision mesh filename=package://justina_description/meshes/robotino/Robotino3_Spl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; visual mesh filename=package://justina_description/meshes/robotino/Robotino3_Whe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
- link wheel1_link: geometry collision mesh filename=package://justina_description/meshes/robotino/Robotino3_Spl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; visual mesh filename=package://justina_description/meshes/robotino/Robotino3_Whe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
- link wheel2_link: geometry collision mesh filename=package://justina_description/meshes/robotino/Robotino3_Spl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; visual mesh filename=package://justina_description/meshes/robotino/Robotino3_Whe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
