Commit message: Fix gripper names

File: urdf/justina.urdf (robot description, URDF)
Before this commit: robot justina, 35 links, 34 joints
Links:
- removed link left_griper_L_link
- removed link left_griper_R_link
- removed link right_griper_L_link
- removed link right_griper_R_link
- added link left_gripper_L_link, mass 0.05; collision mesh filename=package://justina_description/meshes/justina/arm/Gripper_Co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; visual mesh filename=package://justina_description/meshes/justina/arm/Gripper.dae
- added link left_gripper_R_link, mass 0.05; collision mesh filename=package://justina_description/meshes/justina/arm/Gripper_Co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; visual mesh filename=package://justina_description/meshes/justina/arm/Gripper.dae
- added link right_gripper_L_link, mass 0.05; collision mesh filename=package://justina_description/meshes/justina/arm/Gripper_Co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; visual mesh filename=package://justina_description/meshes/justina/arm/Gripper.dae
- added link right_gripper_R_link, mass 0.05; collision mesh filename=package://justina_description/meshes/justina/arm/Gripper_Co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; visual mesh filename=package://justina_description/meshes/justina/arm/Gripper.dae
Joints:
- removed joint left_griper_L_joint
- removed joint left_griper_R_joint
- removed joint right_griper_L_joint
- removed joint right_griper_R_joint
- added joint left_gripper_L_joint: type revolute, parent l_hand_link, child left_gripper_L_link, origin xyz=0 0.01614 -0.169349 rpy=0 0 -1.5708, axis -1 0 0, limit lower=-1.7 upper=1.7 effort=16 velocity=3
- added joint left_gripper_R_joint: type revolute, parent l_hand_link, child left_gripper_R_link, origin xyz=0 -0.01614 -0.169349 rpy=0 0 1.5708, axis 1 0 0, limit lower=-1.7 upper=1.7 effort=16 velocity=3
- added joint right_gripper_L_joint: type revolute, parent r_hand_link, child right_gripper_L_link, origin xyz=0 0.01614 -0.169349 rpy=0 0 -1.5708, axis -1 0 0, limit lower=-1.7 upper=1.7 effort=16 velocity=3
- added joint right_gripper_R_joint: type revolute, parent r_hand_link, child right_gripper_R_link, origin xyz=0 -0.01614 -0.169349 rpy=0 0 1.5708, axis 1 0 0, limit lower=-1.7 upper=1.7 effort=16 velocity=3

Commit message: Add new grippers to urdf and simulation

File: urdf/justina.urdf (robot description, URDF)
Before this commit: robot justina, 35 links, 34 joints
Links:
- added link left_grab_object_link
- added link right_grab_object_link
Joints:
- added joint left_grab_joint: type fixed, parent l_hand_link, child left_grab_object_link, origin xyz=-0.019943 0 -0.2542 rpy=0 0 0
- added joint right_grab_joint: type fixed, parent r_hand_link, child right_grab_object_link, origin xyz=-0.019943 0 -0.2542 rpy=0 0 0

Commit message: Update URDF new arms, set new config in configuring_robot.wbt

File: urdf/justina.urdf (robot description, URDF)
Before this commit: robot justina, 36 links, 35 joints
Links:
- added link left_pinch_object_link
- added link right_pinch_object_link
Joints:
- added joint left_pinch_joint: type fixed, parent l_hand_link, child left_pinch_object_link, origin xyz=-0.005904 0 -0.267347 rpy=0 0 0
- added joint right_pinch_joint: type fixed, parent r_hand_link, child right_pinch_object_link, origin xyz=-0.005904 0 -0.267347 rpy=0 0 0
- joint l_arm_twist_joint: origin xyz=0 0 -0.15 rpy=0 0 0 -> xyz=0 0 -0.09 rpy=0 0 0
- joint l_elbow_joint: origin xyz=0 0 -0.1 rpy=0 0 0 -> xyz=0 0 -0.07 rpy=0 0 0
- joint l_hand_joint: origin xyz=0 0 -0.1 rpy=0 0 0 -> xyz=0 0 -0.07 rpy=0 0 0
- joint l_wrist_joint: origin xyz=0 0 -0.15 rpy=0 0 0 -> xyz=0 0 -0.09 rpy=0 0 0
- joint left_grab_joint: origin xyz=-0.019943 0 -0.2542 rpy=0 0 0 -> xyz=-0.005904 0 -0.237746 rpy=0 0 0
- joint left_gripper_L_joint: origin xyz=0 0.01614 -0.169349 rpy=0 0 -1.5708 -> xyz=-0.005904 0.01614 -0.13759 rpy=0 0 -1.5708
- joint left_gripper_R_joint: origin xyz=0 -0.01614 -0.169349 rpy=0 0 1.5708 -> xyz=-0.005904 -0.01614 -0.13759 rpy=0 0 1.5708
- joint r_arm_twist_joint: origin xyz=0 0 -0.15 rpy=0 0 0 -> xyz=0 0 -0.09 rpy=0 0 0
- joint r_elbow_joint: origin xyz=0 0 -0.1 rpy=0 0 0 -> xyz=0 0 -0.07 rpy=0 0 0
- joint r_hand_joint: origin xyz=0 0 -0.1 rpy=0 0 0 -> xyz=0 0 -0.07 rpy=0 0 0
- joint r_wrist_joint: origin xyz=0 0 -0.15 rpy=0 0 0 -> xyz=0 0 -0.09 rpy=0 0 0
- joint right_grab_joint: origin xyz=-0.019943 0 -0.2542 rpy=0 0 0 -> xyz=-0.005904 0 -0.237746 rpy=0 0 0
- joint right_gripper_L_joint: origin xyz=0 0.01614 -0.169349 rpy=0 0 -1.5708 -> xyz=-0.005904 0.01614 -0.13759 rpy=0 0 -1.5708
- joint right_gripper_R_joint: origin xyz=0 -0.01614 -0.169349 rpy=0 0 1.5708 -> xyz=-0.005904 -0.01614 -0.13759 rpy=0 0 1.5708

Commit message: pinch is grab child

File: urdf/justina.urdf (robot description, URDF)
Before this commit: robot justina, 38 links, 37 joints
Joints:
- joint left_pinch_joint: origin xyz=-0.005904 0 -0.267347 rpy=0 0 0 -> xyz=0 0 -0.029601 rpy=0 0 0; parent l_hand_link -> left_grab_object_link
- joint right_pinch_joint: origin xyz=-0.005904 0 -0.267347 rpy=0 0 0 -> xyz=0 0 -0.029601 rpy=0 0 0; parent r_hand_link -> right_grab_object_link

Commit message: Fix gripper joints axis

File: urdf/justina.urdf (robot description, URDF)
Before this commit: robot justina, 38 links, 37 joints
Joints:
- joint left_gripper_L_joint: axis -1 0 0 -> 0 1 0
- joint left_gripper_R_joint: axis 1 0 0 -> 0 1 0
- joint right_gripper_L_joint: axis -1 0 0 -> 0 1 0
- joint right_gripper_R_joint: axis 1 0 0 -> 0 1 0

Commit message: Update Face_Frame position

File: urdf/justina.urdf (robot description, URDF)
Before this commit: robot justina, 38 links, 37 joints
Joints:
- joint camera_fixed_joint: origin xyz=0 0 0.108729 rpy=-1.5707 0 -1.5707 -> xyz=0 0 0.088981 rpy=-1.5707 0 -1.5707

Commit message: urdf joint limits fixed

File: urdf/justina.urdf (robot description, URDF)
Before this commit: robot justina, 38 links, 37 joints
Joints:
- joint head_pan_joint: limit lower=-1.7 upper=1.7 effort=16 velocity=3 -> lower=-1.57 upper=1.57 effort=16 velocity=3
- joint head_tilt_joint: limit lower=-1.7 upper=1.7 effort=16 velocity=3 -> lower=-1.57 upper=1.57 effort=16 velocity=3
- joint l_arm_twist_joint: limit lower=-1.7 upper=1.7 effort=16 velocity=3 -> lower=-1.57 upper=1.57 effort=16 velocity=3
- joint l_elbow_joint: limit lower=-1.7 upper=1.7 effort=16 velocity=3 -> lower=-1.57 upper=1.57 effort=16 velocity=3
- joint l_hand_joint: limit lower=-1.7 upper=1.7 effort=16 velocity=3 -> lower=-1.57 upper=1.57 effort=16 velocity=3
- joint l_wrist_joint: limit lower=-1.7 upper=1.7 effort=16 velocity=3 -> lower=-1.57 upper=1.57 effort=16 velocity=3
- joint left_grab_joint: origin xyz=-0.005904 0 -0.237746 rpy=0 0 0 -> xyz=-0.005904 0 -0.247746 rpy=0 0 0
- joint left_gripper_L_joint: limit lower=-1.7 upper=1.7 effort=16 velocity=3 -> lower=-1.57 upper=1.57 effort=16 velocity=3
- joint left_gripper_R_joint: limit lower=-1.7 upper=1.7 effort=16 velocity=3 -> lower=-1.57 upper=1.57 effort=16 velocity=3
- joint lf_shoulder_joint: limit lower=-1.7 upper=1.7 effort=16 velocity=3 -> lower=-1.57 upper=1.57 effort=16 velocity=3
- joint ls_shoulder_joint: limit lower=-1.7 upper=1.7 effort=16 velocity=3 -> lower=-1.57 upper=1.57 effort=16 velocity=3
- joint r_arm_twist_joint: limit lower=-1.7 upper=1.7 effort=16 velocity=3 -> lower=-1.57 upper=1.57 effort=16 velocity=3
- joint r_elbow_joint: limit lower=-1.7 upper=1.7 effort=16 velocity=3 -> lower=-1.57 upper=1.57 effort=16 velocity=3
- joint r_hand_joint: limit lower=-1.7 upper=1.7 effort=16 velocity=3 -> lower=-1.57 upper=1.57 effort=16 velocity=3
- joint r_wrist_joint: limit lower=-1.7 upper=1.7 effort=16 velocity=3 -> lower=-1.57 upper=1.57 effort=16 velocity=3
- joint rf_shoulder_joint: limit lower=-1.7 upper=1.7 effort=16 velocity=3 -> lower=-1.57 upper=1.57 effort=16 velocity=3
- joint right_grab_joint: origin xyz=-0.005904 0 -0.237746 rpy=0 0 0 -> xyz=-0.005904 0 -0.247746 rpy=0 0 0
- joint right_gripper_L_joint: limit lower=-1.7 upper=1.7 effort=16 velocity=3 -> lower=-1.57 upper=1.57 effort=16 velocity=3
- joint right_gripper_R_joint: limit lower=-1.7 upper=1.7 effort=16 velocity=3 -> lower=-1.57 upper=1.57 effort=16 velocity=3
- joint rs_shoulder_joint: limit lower=-1.7 upper=1.7 effort=16 velocity=3 -> lower=-1.57 upper=1.57 effort=16 velocity=3

Commit message: moved grab

File: urdf/justina.urdf (robot description, URDF)
Before this commit: robot justina, 38 links, 37 joints
Joints:
- joint left_grab_joint: origin xyz=-0.005904 0 -0.247746 rpy=0 0 0 -> xyz=-0.005904 0 -0.267746 rpy=0 0 0
- joint right_grab_joint: origin xyz=-0.005904 0 -0.247746 rpy=0 0 0 -> xyz=-0.005904 0 -0.267746 rpy=0 0 0

Commit message: Change grippers to simple model

File: urdf/justina.urdf (robot description, URDF)
Before this commit: robot justina, 38 links, 37 joints
Links:
- link left_gripper_L_link: geometry collision mesh filename=package://justina_description/meshes/justina/arm/Gripper_L.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; visual mesh filename=package://justina_description/meshes/justina/arm/Gripper_L.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
- link left_gripper_R_link: geometry collision mesh filename=package://justina_description/meshes/justina/arm/Gripper_R.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; visual mesh filename=package://justina_description/meshes/justina/arm/Gripper_R.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
- link right_gripper_L_link: geometry collision mesh filename=package://justina_description/meshes/justina/arm/Gripper_L.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; visual mesh filename=package://justina_description/meshes/justina/arm/Gripper_L.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
- link right_gripper_R_link: geometry collision mesh filename=package://justina_description/meshes/justina/arm/Gripper_R.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; visual mesh filename=package://justina_description/meshes/justina/arm/Gripper_R.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
Joints:
- joint left_gripper_L_joint: origin xyz=-0.005904 0.01614 -0.13759 rpy=0 0 -1.5708 -> xyz=-0.005904 0.01614 -0.13759 rpy=0 0 0
- joint left_gripper_R_joint: origin xyz=-0.005904 -0.01614 -0.13759 rpy=0 0 1.5708 -> xyz=-0.005904 -0.01614 -0.13759 rpy=0 0 0
- joint right_gripper_L_joint: origin xyz=-0.005904 0.01614 -0.13759 rpy=0 0 -1.5708 -> xyz=-0.005904 0.01614 -0.13759 rpy=0 0 0
- joint right_gripper_R_joint: origin xyz=-0.005904 -0.01614 -0.13759 rpy=0 0 1.5708 -> xyz=-0.005904 -0.01614 -0.13759 rpy=0 0 0

Commit message: Fix grippers motion axis

File: urdf/justina.urdf (robot description, URDF)
Before this commit: robot justina, 38 links, 37 joints
Joints:
- joint left_gripper_L_joint: axis 0 1 0 -> 1 0 0
- joint left_gripper_R_joint: axis 0 1 0 -> -1 0 0
- joint right_gripper_L_joint: axis 0 1 0 -> 1 0 0
- joint right_gripper_R_joint: axis 0 1 0 -> -1 0 0

Commit message: Fix pinch & grasp links

File: urdf/justina.urdf (robot description, URDF)
Before this commit: robot justina, 38 links, 37 joints
Joints:
- joint left_grab_joint: origin xyz=-0.005904 0 -0.267746 rpy=0 0 0 -> xyz=-0.005904 0 -0.237746 rpy=0 0 0
- joint right_grab_joint: origin xyz=-0.005904 0 -0.267746 rpy=0 0 0 -> xyz=-0.005904 0 -0.237746 rpy=0 0 0

Commit message: modificated urdf and add xtion launch

File: urdf/justina.urdf (robot description, URDF)
Before this commit: robot justina, 38 links, 37 joints
Joints:
- joint camera_fixed_joint: origin xyz=0 0 0.088981 rpy=-1.5707 0 -1.5707 -> xyz=0 0 0.088981 rpy=0 0 0

Commit message: URDF grippers fixed

File: urdf/justina.urdf (robot description, URDF)
Before this commit: robot justina, 38 links, 37 joints
Joints:
- joint left_grab_joint: origin xyz=-0.005904 0 -0.237746 rpy=0 0 0 -> xyz=-0.005904 0 -0.23 rpy=0 0 0
- joint left_pinch_joint: origin xyz=0 0 -0.029601 rpy=0 0 0 -> xyz=0 0 -0.04 rpy=0 0 0
- joint right_grab_joint: origin xyz=-0.005904 0 -0.237746 rpy=0 0 0 -> xyz=-0.005904 0 -0.23 rpy=0 0 0
- joint right_pinch_joint: origin xyz=0 0 -0.029601 rpy=0 0 0 -> xyz=0 0 -0.04 rpy=0 0 0
