Commit message: Add xtion mesh, set urdf camera position

File: urdf/justina.urdf (robot description, URDF)
Before this commit: robot justina, 38 links, 37 joints
Links:
- link camera_link: geometry collision mesh filename=package://justina_description/meshes/justina/face/Xtion_Col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; visual mesh filename=package://justina_description/meshes/justina/face/Xtion.dae
Joints:
- joint camera_fixed_joint: origin xyz=0 0 0.088981 rpy=0 0 0 -> xyz=0 0 0.1275 rpy=-1.5707 0 -1.5707

Commit message: Original frame orientation except visual model

File: urdf/justina.urdf (robot description, URDF)
Before this commit: robot justina, 38 links, 37 joints
Joints:
- joint camera_fixed_joint: origin xyz=0 0 0.1275 rpy=-1.5707 0 -1.5707 -> xyz=0 0 0.1275 rpy=0 0 0

Commit message: Z fixed

File: urdf/justina.urdf (robot description, URDF)
Before this commit: robot justina, 38 links, 37 joints
Joints:
- joint camera_fixed_joint: origin xyz=0 0 0.1275 rpy=0 0 0 -> xyz=0 0 0.108 rpy=0 0 0

Commit message: offset in camera_color_optical_frame

File: urdf/justina.urdf (robot description, URDF)
Before this commit: robot justina, 38 links, 37 joints
Joints:
- joint camera_fixed_joint: origin xyz=0 0 0.108 rpy=0 0 0 -> xyz=0 0.0225 0.108 rpy=0 0 0
